File: MST01.kicad_pcb (KiCad board)
At the start: 4 copper layers, 108.8 x 76.9 mm, 139 parts, among them J1 Conn_01x35, J2 Conn_01x35, J3 Conn_01x04_Pin, J6 Conn_01x05, J8 USB_B_Mini, M1 Module-power_12and5V-0.2, M2 Module-knock-0.2, M3 Module-vr-discrete-0.5, M4 Module-vr-max9924-0.1, M5 Module-wbo-0.5, M6 Module:mega-mcu100/0.3, M7 Module-can-0.1, P1 Pad, P10 Pad, P15 Pad, P16 Pad, P17 Pad, P18 Pad, P2 Pad, P3 Pad, P4 Pad, P5 Pad, P6 Pad, P7 Pad, P8 Pad, P9 Pad, Q10 ISL9V3040D3ST, Q11 ISL9V3040D3ST, Q12 ISL9V3040D3ST, Q7 ISL9V3040D3ST, Q8 ISL9V3040D3ST, Q9 ISL9V3040D3ST, U1 TLE9201SG, U10 VNLD5160TR-E, U11 VNLD5160TR-E, U12 MPXH6400A, U2 TLE9201SG, U4 MAX31855KASA, U5 JDY-33-mio, U6 VNLD5160TR-E, U7 VNLD5160TR-E, U8 VNLD5160TR-E, U9 VNLD5160TR-E

Commit message: Aggiornamento PCB
Parts:
- G2: moved to B.Cu
- moved G2 572.9 mm to (165.3, 139.1), turned to 180 degrees
- moved M4 0.10 mm to (180.0, 108.5)
- moved M3 0.08 mm to (180.0, 130.5)
Routing:
- net +3.3V: track 104.9 -> 109.6 mm
- net +3.3VA: track 195.3 -> 197.0 mm
- net /VMAIN: track 88.4 -> 86.7 mm
- net /CAN1-: track 116.9 -> 116.2 mm
- net /IMP_VR_MAX9924+: track 19.2 -> 19.7 mm
- net Net-(M6-UART2_RX_(PD6)): track 31.4 -> 31.9 mm
- net GND: vias 223 -> 233
Other:
- board text added: "MST01 rev.A"

Commit message: Aggiornamento
Parts:
- moved G1 580.4 mm to (151.8, 82.5)
- moved D1 10.3 mm to (123.6, 138.2), turned to -90 degrees
- moved J3 0.40 mm to (121.8, 139.2)
- moved F6 0.32 mm to (84.7, 71.7)
- moved F5 0.30 mm to (76.3, 82.1)
- moved BT1 0.10 mm to (134.7, 138.0)
Connections:
- net Net-(J1-Pin_26) renamed /P10
- net Net-(J1-Pin_31) renamed /P9
- net Net-(J2-Pin_32) renamed /P1
- net Net-(J2-Pin_33) renamed /P2
- net Net-(J6-Pin_1) renamed /V33_OUT
- net Net-(J6-Pin_2) renamed /SWCLK
- net Net-(J6-Pin_4) renamed /SWDIO
- net Net-(J6-Pin_5) renamed /nReset
Routing:
- net +3.3VA: track 197.0 -> 190.6 mm
- net Net-(BT1-+): track 7.06 -> 3.67 mm
- net Net-(M6-SPI2_CS_/_CAN2_RX_(PB12)): track 73.0 -> 71.4 mm
- net /WBO_Rtrim: track 31.9 -> 33.0 mm
- net /VBAT: track 50.4 -> 51.0 mm, vias 5 -> 6
- net GNDA: track 67.0 -> 66.5 mm
Other:
- board text added: "+12V"
- board text added: "+3.3VA"
- board text added: "+5V"
- board text added: "+5VA"
- board text added: "12V_KEY"
- board text added: "CAN1+"
- board text added: "CAN1-"
- board text added: "CAN2+"
- board text added: "CAN2-"
- board text added: "D+"
- board text added: "D-"
- board text added: "EGT+"
- board text added: "EGT-"
- board text added: "P1"
- board text added: "P10"
- board text added: "P2"
- board text added: "P9"
- board text added: "UART2 TX RX"
- board text added: "V33_OUT SWCLK GND SWDIO nReset"
- board text added: "VR9924+"
- board text added: "VR9924-"
- board text added: "VRDis+"
- board text added: "VRDis-"
- board text added: "Vbus"
- board text added: "WB_Header"
- board text added: "WB_Ip"
- board text added: "WB_Rtrim"
- board text added: "WB_Un"
- board text added: "WB_Vm"
- board text removed: "+ EGT -"
- board text removed: "1"
- board text removed: "10"
- board text removed: "11"
- board text removed: "12"
- board text removed: "12V"
- board text removed: "16"
- board text removed: "18"
- board text removed: "20"
- board text removed: "3"
- board text removed: "3.3"
- board text removed: "4"
- board text removed: "5"
- board text removed: "5V"
- board text removed: "6"
- board text removed: "8"
- board text removed: "9"
- board text removed: "9924+"
- board text removed: "9924-"
- board text removed: "A"
- board text removed: "Always looking for C/C++/PHP/Java developers https://rusefi.com/s/mission"
- board text removed: "B"
- board text removed: "C"
- board text removed: "CAN2"
- board text removed: "COMMUNITY SUPPORT ECU"
- board text removed: "D"
- board text removed: "DISCRETE+"
- board text removed: "DISCRETE-"
- board text removed: "E"
- board text removed: "G"
- board text removed: "G G + - V"
- board text removed: "H CAN L"
- board text removed: "Heater"
- board text removed: "Ignition logic level outputs by default to control dumb coils remove R20-R22, R26-R28 and populate Q7-Q12"
- board text removed: "Ip"
- board text removed: "L CAN H"
- board text removed: "Rtrim"
- board text removed: "SWD: R D G C V"
- board text removed: "To enable Hall mode on VR9924-, populate R1"
- board text removed: "UAEFI rev. D"
- board text removed: "UART2 RX TX"
- board text removed: "USB"
- board text removed: "Un"
- board text removed: "VIGN"
- board text removed: "VR 9924 DISCR"
- board text removed: "Vm"
- board text removed: "WBO"
- board text removed: "https://rusefi.com/s/uaefi"

Commit message: Aggiornamento Progetto
Parts:
- J1, J2: value Conn_01x35 -> Conn_01x36; footprint ampseal:ampseal-35-mia -> ampseal:ampseal-35-mia-con-pad-GND
- moved R3 1.04 mm to (92.6, 137.3)
- moved R2 0.97 mm to (97.0, 137.3)
- moved R6 0.63 mm to (159.4, 76.9), turned to 180 degrees
Routing:
- net +3.3V: track 109.6 -> 101.6 mm
- net +5VA: track 174.5 -> 178.2 mm
- net /VMAIN: track 86.7 -> 88.5 mm
- net /ADC3: track 69.5 -> 68.1 mm
- net Net-(M6-SPI2_SCK_/_CAN2_TX_(PB13)): track 75.6 -> 75.1 mm
- net GND: vias 233 -> 207
- net /WBO_Ip: vias 0 -> 1
- net /OUT_LS_HOT2: vias 0 -> 1

Commit message: Aggiornamento PCB
Parts:
- C1, C10, C11, C14, C15, C16, C17, C18, C19, C2, C20, C21, C22, C23, C24, C3, C4, C5, C6, C7, C8, C9, F10, F5, F6, F7, F8, F9, R17, R18, R19, R20, R21, R22, R23, R24, R25, R26: moved to F.Cu
- C12, C13, C25, C26, Q11, Q12, R14, R9, U1, U2: moved to B.Cu
- J1, J2: value Conn_01x36 -> DNP
- J6: value Conn_01x05 -> DNP
- P1, P2, P3, P4, P5, P6, P7, P8, P9: value Pad -> DNP
- P10, P15, P16, P17, P18: value Pad -> DNP; footprint hellen-one-common:PAD-TH -> Impronte-mie:PAD-TH-senza-serigrafia
- Q10, Q7, Q8, Q9: value ISL9V3040D3ST -> DNP; moved to B.Cu
- R1: value 4.7k -> DNP
- R27, R28: value 0 -> DNP; moved to F.Cu
- R5: value 0 -> DNP
- moved C18 19.4 mm to (83.5, 141.8)
- moved C23 19.4 mm to (87.5, 141.8)
- moved C6 19.3 mm to (78.9, 124.8)
- moved C1 19.3 mm to (74.9, 124.8)
- moved C2 15.9 mm to (74.9, 126.8)
- moved C7 15.9 mm to (78.9, 126.8)
- moved C22 15.8 mm to (87.5, 139.8)
- moved C17 15.8 mm to (83.5, 139.7)
- moved C11 12.9 mm to (75.0, 134.1)
- moved R14 12.9 mm to (80.7, 143.2), turned to 180 degrees
- moved C3 12.8 mm to (74.9, 128.8)
- moved C8 12.8 mm to (78.9, 128.8)
- moved U1 12.7 mm to (76.4, 128.8), turned to -90 degrees
- moved U2 12.7 mm to (85.0, 137.8), turned to -90 degrees
- moved C24 12.6 mm to (83.6, 143.2)
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Connections:
- net Net-(U4-T+) renamed /EGT/T+Filtrato
- net Net-(U4-T-) renamed /EGT/T-Filtrato
- J1 pad 1: /OUT_DC2- -> /OUT_DC1+
- J1 pad 13: /OUT_DC1- -> /OUT_DC2+
- J1 pad 14: /OUT_DC1+ -> /OUT_DC2-
- J1 pad 2: /OUT_DC2+ -> /OUT_DC1-
- J1 pad 32: /OUT_IGN3 -> GND
- J1 pad 33: GND -> /OUT_IGN3
Routing:
- net /IGN2: track 107.5 -> 130.0 mm
- net /DC1_DIS: track 91.5 -> 72.3 mm
- net +3.3V: track 101.6 -> 119.2 mm, vias 2 -> 8
- net +5VA: track 178.2 -> 163.1 mm
- net /OUT_DC2+: track 5.74 -> 19.1 mm
- net /OUT_DC1-: track 20.0 -> 7.86 mm
- net /DC2_DIS: track 71.9 -> 60.6 mm
- net /DC1_DIR: track 69.7 -> 59.6 mm, vias 4 -> 3
- net /DC1_PWM: track 63.9 -> 72.3 mm, vias 4 -> 2
- net /P9: track 9.31 -> 17.1 mm
- net /DC2_PWM: track 58.2 -> 65.7 mm, vias 4 -> 2
- net /CAN1+: track 110.9 -> 118.2 mm
- net /CAN1-: track 116.2 -> 122.9 mm
- net /DC Driver 1/PWR: track 17.2 -> 22.2 mm
- net /IGN1: track 109.6 -> 113.7 mm
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- added copper zone on F.Cu, net /DC Driver 1/PWR
- added copper zone on F.Cu, net /DC Driver 2/PWR
- added copper zone on F.Cu, net /OUT_IGN1
- added copper zone on F.Cu, net /OUT_IGN2
- added copper zone on F.Cu, net /OUT_IGN3
- added copper zone on F.Cu, net /OUT_IGN4
- added copper zone on F.Cu, net /OUT_IGN5
- added copper zone on F.Cu, net /OUT_IGN6
- removed copper zone on B.Cu, net /DC Driver 1/PWR
- removed copper zone on B.Cu, net /DC Driver 2/PWR
- removed copper zone on B.Cu, net /OUT_IGN1
- removed copper zone on B.Cu, net /OUT_IGN2
- removed copper zone on B.Cu, net /OUT_IGN3
- removed copper zone on B.Cu, net /OUT_IGN4
- removed copper zone on B.Cu, net /OUT_IGN5
- removed copper zone on B.Cu, net /OUT_IGN6
Other:
- board text added: "1"
- board text added: "2"
- board text added: "LS"
