File: MST01.kicad_pcb (KiCad board)
At the start: 4 copper layers, 108.8 x 76.9 mm, 139 parts, among them J1 DNP, J2 DNP, J3 Conn_01x04_Pin, J6 DNP, J8 USB_B_Mini, M1 Module-power_12and5V-0.2, M2 Module-knock-0.2, M3 Module-vr-discrete-0.5, M4 Module-vr-max9924-0.1, M5 Module-wbo-0.5, M6 Module:mega-mcu100/0.3, M7 Module-can-0.1, P1 DNP, P10 DNP, P15 DNP, P16 DNP, P17 DNP, P18 DNP, P2 DNP, P3 DNP, P4 DNP, P5 DNP, P6 DNP, P7 DNP, P8 DNP, P9 DNP, Q10 DNP, Q11 ISL9V3040D3ST, Q12 ISL9V3040D3ST, Q7 DNP, Q8 DNP, Q9 DNP, U1 TLE9201SG, U10 VNLD5160TR-E, U11 VNLD5160TR-E, U12 MPXH6400A, U2 TLE9201SG, U4 MAX31855KASA, U5 JDY-33-mio, U6 VNLD5160TR-E, U7 VNLD5160TR-E, U8 VNLD5160TR-E, U9 VNLD5160TR-E

Commit message: Aggiornamento Progetto
Parts:
- J1: value DNP -> AMPSeal-35-verticale-nero
- J2: value DNP -> AMPSeal-35-verticale-bianco
- J6: value DNP -> Conn_01x05_Pin
- P1, P10, P15, P16, P17, P18, P2, P3, P4, P5, P6, P7, P8, P9: value DNP -> Pad
- Q10, Q7, Q8, Q9: value DNP -> ISL9V3040D3ST
- R1: value DNP -> 4.7k
- R27, R28, R5: value DNP -> 0
- R38, R39, R40: value DNP -> 10k
- U5: value JDY-33-mio -> JDY-33
Routing:
- net /PWR_EN: track 42.4 -> 43.9 mm

Commit message: Aggiornamento Progetto
Parts:
- removed P16, P18: Pad, Impronte-mie:PAD-TH-senza-serigrafia
- removed R14: 4.7k, hellen-one-common:R0603
- added P11: Pad, Impronte-mie:PAD-TH-senza-serigrafia, F.Cu at (112.4, 116.3)
- added P12: Pad, Impronte-mie:PAD-TH-senza-serigrafia, F.Cu at (111.0, 118.4)
- added R7: 4.7k, hellen-one-common:R0603, B.Cu at (80.7, 143.7)
- moved P7 0.63 mm to (150.4, 127.9)
- moved C26 0.33 mm to (88.4, 130.8)
- moved C17 0.07 mm to (83.5, 139.8)
Connections:
- net /DC Driver 1/PWR renamed /2 DC Driver/PWR1
- net /DC Driver 2/PWR renamed /2 DC Driver/PWR2
Routing:
- net /DC2_DIR: track 75.2 -> 76.1 mm
- net Net-(M6-LED_GREEN): track 3.75 -> 4.64 mm
- net Net-(M6-UART2_RX_(PD6)): track 31.9 -> 32.7 mm
- net /VR_DISCRETE: track 52.1 -> 51.6 mm
- net GND: vias 210 -> 216
Other:
- board text removed: "1"
- board text removed: "2"
- board text removed: "LS"

Commit message: MST01-a1
Changed lines of the file:
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@@
 			)
 		)
-		(property "LCSC" ""
+		(property "LCSC" "C25469"
 			(at 0 0 180)
 			(unlocked yes)
@@
 			)
 		)
-		(property "MyComment" "C25469"
+		(property "MyComment" ""
 			(at 0 0 0)
 			(unlocked yes)
@@
 			)
 		)
-		(property "Note-mie" "DNP"
+		(property "Note-mie" ""
 			(at 0 0 180)
 			(unlocked yes)
@@
 		(tags "fuse")
 		(property "Reference" "F6"
-			(at 0.41625 -2.1225 180)
+			(at -0.03 -3.27 180)
 			(layer "F.SilkS")
 			(effects
@@
 			)
 		)
-		(property "MyComment" "776231-4    Aliexpress"
+		(property "MyComment" "Aliexpress"
 			(at 0 0 -90)
 			(unlocked yes)
@@
 			)
 		)
-		(property "LCSC" ""
+		(property "LCSC" "776231-4"
 			(at 0 0 -90)
 			(unlocked yes)
@@
 			)
 		)
-		(property "Note-mie" "DNP"
+		(property "Note-mie" ""
 			(at 0 0 -90)
 			(unlocked yes)
@@
 		(at 73.43 95.08 180)
 		(property "Reference" "R15"
-			(at 1.26 0.89 0)
+			(at 1.21 1.9 0)
 			(unlocked yes)
 			(layer "F.SilkS")
@@
 		(at 81.08 71.9 -90)
 		(property "Reference" "R17"
-			(at 2.49 1.12 0)
+			(at -0.71 -2.62 0)
 			(unlocked yes)
 			(layer "F.SilkS")
@@
 		(tags "fuse")
 		(property "Reference" "F5"
-			(at 0.19375 -1.63 180)
+			(at 0.83 -3.01 180)
 			(layer "F.SilkS")
 			(effects
@@
 		(at 75 82.13 -90)
 		(property "Reference" "R18"
-			(at 2.48 1.095 0)
+			(at 0.29 -2.36 0)
 			(unlocked yes)
 			(layer "F.SilkS")
@@
 		(tags "resistor")
 		(property "Reference" "R20"
-			(at 1.21 3.31 180)
+			(at 0.43 3.59 180)
 			(layer "F.SilkS")
 			(effects
@@
 			)
 		)
-		(property "LCSC" ""
-			(at 0 0 -90)
-			(unlocked yes)
-			(layer "F.Fab")
-			(hide yes)
-			(effects
-				(font
-					(size 1 1)
-					(thickness 0.15)
-				)
-			)
-		)
-		(property "MyComment" "C9900001612   Aliexpress"
+		(property "LCSC" "C9900001612"
 			(at 0 0 -90)
 			(unlocked yes)
@@
 			)
 		)
-		(property "Note-mie" "DNP"
+		(property "MyComment" "Aliexpress"
 			(at 0 0 -90)
 			(unlocked yes)
@@
 			)
 		)
-		(property "MyComment" "Ci sono"
+		(property "MyComment" ""
 			(at 0 0 90)
 			(unlocked yes)
@@
 			)
 		)
-		(property "Note-mie" "DNP"
+		(property "Note-mie" ""
 			(at 0 0 90)
 			(unlocked yes)
@@
 			)
 		)
-		(property "MyComment" "776231-1    Aliexpress"
+		(property "MyComment" "Aliexpress"
 			(at 0 0 90)
 			(unlocked yes)
@@
 			)
 		)
-		(property "LCSC" ""
+		(property "LCSC" "776231-1"
 			(at 0 0 90)
 			(unlocked yes)
@@
 			)
 		)
-		(property "Note-mie" "DNP"
+		(property "Note-mie" ""
 			(at 0 0 90)
 			(unlocked yes)
@@
 			)
 		)
-		(property "LCSC" ""
+		(property "LCSC" "C25469"
 			(at 0 0 180)
 			(unlocked yes)
@@
 			)
 		)
-		(property "MyComment" "C25469"
+		(property "MyComment" ""
 			(at 0 0 0)
 			(unlocked yes)
@@
 			)
 		)
-		(property "Note-mie" "DNP"
+		(property "Note-mie" ""
 			(at 0 0 180)
 			(unlocked yes)
@@
 			)
 		)
-		(property "LCSC" ""
+		(property "LCSC" "C17414"
 			(at 0 0 0)
 			(layer "B.Fab")
@@
 			)
 		)
-		(property "MyComment" "C17414"
+		(property "MyComment" ""
 			(at 0 0 180)
 			(unlocked yes)
@@
 			)
 		)
-		(property "Note-mie" "DNP"
+		(property "Note-mie" ""
 			(at 0 0 180)
 			(unlocked yes)
@@
 			)
 		)
-		(property "LCSC" ""
+		(property "LCSC" "C17414"
 			(at 0 0 0)
 			(layer "B.Fab")
@@
 			)
 		)
-		(property "MyComment" "C17414"
+		(property "MyComment" ""
 			(at 0 0 180)
 			(unlocked yes)
@@
 			)
 		)
-		(property "Note-mie" "DNP"
+		(property "Note-mie" ""
 			(at 0 0 180)
 			(unlocked yes)
@@
 			)
 		)
-		(property "LCSC" ""
+		(property "LCSC" "C462128"
 			(at 145.32 -209 90)
 			(layer "B.Fab")
@@
 			)
 		)
-		(property "MyComment" "C462128"
+		(property "MyComment" ""
 			(at 145.32 -209 90)
 			(layer "B.Fab")
@@
 			)
 		)
-		(property "Note-mie" "DNP"
+		(property "Note-mie" ""
 			(at 0 0 -90)
 			(unlocked yes)
@@
 			)
 		)
-		(property "LCSC" ""
+		(property "LCSC" "C23162"
 			(at 169.864994 -160.15 0)
 			(layer "B.Fab")
@@
 			)
 		)
-		(property "MyComment" "C23162"
+		(property "MyComment" ""
 			(at 169.864994 -160.15 0)
 			(layer "B.Fab")
@@
 			)
 		)
-		(property "Note-mie" "DNP"
+		(property "Note-mie" ""
 			(at 0 0 0)
 			(unlocked yes)
@@
 			)
 		)
-		(property "LCSC" ""
+		(property "LCSC" "C462128"
 			(at 0 0 0)
 			(unlocked yes)
@@
 			)
 		)
-		(property "MyComment" "C462128"
+		(property "MyComment" ""
 			(at 0 0 0)
 			(unlocked yes)
@@
 			)
 		)
-		(property "Note-mie" "DNP"
+		(property "Note-mie" ""
 			(at 0 0 180)
 			(unlocked yes)
@@
 			)
 		)
-		(property "LCSC" ""
+		(property "LCSC" "C2653438"
 			(at 0 0 90)
 			(unlocked yes)
@@
 			)
 		)
-		(property "MyComment" "C2653438"
+		(property "MyComment" "Aliexpress"
 			(at 0 0 -90)
 			(unlocked yes)
@@
 			)
 		)
-		(property "Note-mie" "DNP"
+		(property "Note-mie" ""
 			(at 0 0 -90)
 			(unlocked yes)
@@
 			)
 		)
-		(property "LCSC" ""
+		(property "LCSC" "C17414"
 			(at 0 0 0)
 			(layer "B.Fab")
@@
 			)
 		)
-		(property "MyComment" "C17414"
+		(property "MyComment" ""
 			(at 0 0 180)
 			(unlocked yes)
@@
 			)
 		)
-		(property "Note-mie" "DNP"
+		(property "Note-mie" ""
 			(at 0 0 180)
 			(unlocked yes)
@@
 			)
 		)
-		(property "LCSC" ""
+		(property "LCSC" "C462128"
 			(at 0 0 0)
 			(unlocked yes)
@@
 			)
 		)
-		(property "MyComment" "C462128"
+		(property "MyComment" ""
 			(at 0 0 0)
 			(unlocked yes)
@@
 			)
 		)
-		(property "Note-mie" "DNP"
+		(property "Note-mie" ""
 			(at 0 0 180)
 			(unlocked yes)
@@
 			)
 		)
-		(property "MyComment" ""
+		(property "MyComment" "Aliexpress"
 			(at 0 0 90)
 			(unlocked yes)
@@
 			)
 		)
-		(property "LCSC" ""
+		(property "LCSC" "C21189"
 			(at 8.7 205.1 0)
 			(layer "B.Fab")
@@
 			)
 		)
-		(property "MyComment" "C21189"
+		(property "MyComment" ""
 			(at 8.7 205.1 0)
 			(layer "B.Fab")
@@
 			)
 		)
-		(property "Note-mie" "DNP"
+		(property "Note-mie" ""
 			(at 0 0 90)
 			(unlocked yes)
@@
 			)
 		)
-		(property "LCSC" ""
+		(property "LCSC" "C462128"
 			(at 0 0 90)
 			(unlocked yes)
@@
 			)
 		)
-		(property "MyComment" "C462128"
+		(property "MyComment" ""
 			(at 0 0 90)
 			(unlocked yes)
@@
 			)
 		)
-		(property "Note-mie" "DNP"
+		(property "Note-mie" ""
 			(at 0 0 -90)
 			(unlocked yes)

Commit message: MST01-a2
Parts:
- M1: value Module-power_12and5V-0.2 -> Module-power_12and5V-0.3; footprint hellen-one-power_12and5V-0.2:power_12and5V -> hellen-one-power_12and5V-0.3:power_12and5V
