File: MST01.kicad_pcb (KiCad board)
At the start: 4 copper layers, 108.8 x 76.9 mm, 139 parts, among them J1 AMPSeal-35-verticale-nero, J2 AMPSeal-35-verticale-bianco, J3 Conn_01x04_Pin, J6 Conn_01x05_Pin, J8 USB_B_Mini, M1 Module-power_12and5V-0.3, M2 Module-knock-0.2, M3 Module-vr-discrete-0.5, M4 Module-vr-max9924-0.1, M5 Module-wbo-0.5, M6 Module:mega-mcu100/0.3, M7 Module-can-0.1, P1 Pad, P10 Pad, P11 Pad, P12 Pad, P15 Pad, P17 Pad, P2 Pad, P3 Pad, P4 Pad, P5 Pad, P6 Pad, P7 Pad, P8 Pad, P9 Pad, Q10 ISL9V3040D3ST, Q11 ISL9V3040D3ST, Q12 ISL9V3040D3ST, Q7 ISL9V3040D3ST, Q8 ISL9V3040D3ST, Q9 ISL9V3040D3ST, U1 TLE9201SG, U10 VNLD5160TR-E, U11 VNLD5160TR-E, U12 MPXH6400A, U2 TLE9201SG, U4 MAX31855KASA, U5 JDY-33, U6 VNLD5160TR-E, U7 VNLD5160TR-E, U8 VNLD5160TR-E, U9 VNLD5160TR-E

Commit message: MST01-a5
Routing:
- net /OUT_LS1: track 15.1 -> 13.6 mm

Commit message: aggiornamento
Changed lines of the file:
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@@
 		(allow_soldermask_bridges_in_footprints no)
 		(aux_axis_origin 71.345 145.255)
+		(grid_origin 71.345 145.255)
 		(pcbplotparams
 			(layerselection 0x00010fc_ffffffff)
@@
 	)
 	(gr_text "IGN3"
-		(at 90.395 95.58 0)
+		(at 90.385 91.475 0)
 		(layer "F.SilkS")
 		(effects
@@
 	)
 	(gr_text "GND"
-		(at 90.555 91.57 0)
+		(at 90.515 95.385 0)
 		(layer "F.SilkS")
 		(effects
