File: DC_MOTOR_1.kicad_sch (KiCad schematic)
At the start: 17 parts, among them P15 DNP, P17 DNP, U1 TLE9201SG

Commit message: Aggiornamento Progetto
Parts:
- C? (x13), R?: MyComment x -> (none)
- P15, P17: value DNP -> Pad; MyComment x -> (none); now fitted
- U1: LCSC C2653438 -> (none); MyComment x -> C2653438; Note-mie (none) -> DNP; now fitted
Changed lines of the file:
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@@
 			)
 		)
-		(property "MyComment" "x"
+		(property "MyComment" ""
+			(at 127 83.82 0)
+			(effects
+				(font
+					(size 1.27 1.27)
+				)
+				(hide yes)
+			)
+		)
+		(property "Note-mie" ""
 			(at 127 83.82 0)
 			(effects
@@
 			)
 		)
-		(property "MyComment" "x"
+		(property "MyComment" ""
+			(at 109.22 83.82 0)
+			(effects
+				(font
+					(size 1.27 1.27)
+				)
+				(hide yes)
+			)
+		)
+		(property "Note-mie" ""
 			(at 109.22 83.82 0)
 			(effects
@@
 			)
 		)
-		(property "MyComment" "x"
+		(property "MyComment" ""
+			(at 153.67 83.82 0)
+			(effects
+				(font
+					(size 1.27 1.27)
+				)
+				(hide yes)
+			)
+		)
+		(property "Note-mie" ""
 			(at 153.67 83.82 0)
 			(effects
@@
 			)
 		)
-		(property "MyComment" "x"
+		(property "MyComment" ""
+			(at 135.89 83.82 0)
+			(effects
+				(font
+					(size 1.27 1.27)
+				)
+				(hide yes)
+			)
+		)
+		(property "Note-mie" ""
 			(at 135.89 83.82 0)
 			(effects
@@
 			)
 		)
-		(property "MyComment" "x"
+		(property "MyComment" ""
+			(at 175.26 111.76 0)
+			(effects
+				(font
+					(size 1.27 1.27)
+				)
+				(hide yes)
+			)
+		)
+		(property "Note-mie" ""
 			(at 175.26 111.76 0)
 			(effects
@@
 			)
 		)
-		(property "MyComment" "x"
+		(property "MyComment" ""
+			(at 73.66 83.82 0)
+			(effects
+				(font
+					(size 1.27 1.27)
+				)
+				(hide yes)
+			)
+		)
+		(property "Note-mie" ""
 			(at 73.66 83.82 0)
 			(effects
@@
 			)
 		)
-		(property "MyComment" "x"
+		(property "MyComment" ""
+			(at 162.56 83.82 0)
+			(effects
+				(font
+					(size 1.27 1.27)
+				)
+				(hide yes)
+			)
+		)
+		(property "Note-mie" ""
 			(at 162.56 83.82 0)
 			(effects
@@
 			)
 		)
-		(property "MyComment" "x"
+		(property "MyComment" ""
+			(at 100.33 83.82 0)
+			(effects
+				(font
+					(size 1.27 1.27)
+				)
+				(hide yes)
+			)
+		)
+		(property "Note-mie" ""
 			(at 100.33 83.82 0)
 			(effects
@@
 			)
 		)
-		(property "MyComment" "x"
+		(property "MyComment" ""
+			(at 144.78 83.82 0)
+			(effects
+				(font
+					(size 1.27 1.27)
+				)
+				(hide yes)
+			)
+		)
+		(property "Note-mie" ""
 			(at 144.78 83.82 0)
 			(effects
@@
 		(in_bom yes)
 		(on_board yes)
-		(dnp yes)
+		(dnp no)
 		(property "Reference" "P15"
 			(at 222.25 107.95 0)
@@
 			)
 		)
-		(property "Value" "DNP"
+		(property "Value" "Pad"
 			(at 220.98 110.49 0)
 			(effects
@@
 			)
 		)
-		(property "MyComment" "x"
+		(property "MyComment" ""
+			(at 220.98 107.95 0)
+			(effects
+				(font
+					(size 1.27 1.27)
+				)
+				(hide yes)
+			)
+		)
+		(property "Note-mie" ""
 			(at 220.98 107.95 0)
 			(effects
@@
 			)
 		)
-		(property "MyComment" "x"
+		(property "MyComment" ""
+			(at 219.71 101.6 0)
+			(effects
+				(font
+					(size 1.27 1.27)
+				)
+				(hide yes)
+			)
+		)
+		(property "Note-mie" ""
 			(at 219.71 101.6 0)
 			(effects
@@
 		(in_bom yes)
 		(on_board yes)
-		(dnp yes)
+		(dnp no)
 		(fields_autoplaced yes)
 		(property "Reference" "U1"
@@
 			)
 		)
-		(property "LCSC" "C2653438"
+		(property "LCSC" ""
 			(at 198.12 93.98 0)
 			(effects
@@
 			)
 		)
-		(property "MyComment" "x"
+		(property "MyComment" "C2653438"
 			(at 198.12 93.98 0)
 			(effects
@@
 				)
 				(hide yes)
+			)
+		)
+		(property "Note-mie" "DNP"
+			(at 198.12 93.98 0)
+			(effects
+				(font
+					(size 1.27 1.27)
+				)
 			)
 		)
@@
 			)
 		)
-		(property "MyComment" "x"
+		(property "MyComment" ""
+			(at 118.11 83.82 0)
+			(effects
+				(font
+					(size 1.27 1.27)
+				)
+				(hide yes)
+			)
+		)
+		(property "Note-mie" ""
 			(at 118.11 83.82 0)
 			(effects
@@
 			)
 		)
-		(property "MyComment" "x"
+		(property "MyComment" ""
+			(at 175.26 92.71 0)
+			(effects
+				(font
+					(size 1.27 1.27)
+				)
+				(hide yes)
+			)
+		)
+		(property "Note-mie" ""
 			(at 175.26 92.71 0)
 			(effects
@@
 		(in_bom yes)
 		(on_board yes)
-		(dnp yes)
+		(dnp no)
 		(property "Reference" "P17"
 			(at 222.25 105.41 0)
@@
 			)
 		)
-		(property "Value" "DNP"
+		(property "Value" "Pad"
 			(at 220.98 107.95 0)
 			(effects
@@
 			)
 		)
-		(property "MyComment" "x"
+		(property "MyComment" ""
+			(at 220.98 105.41 0)
+			(effects
+				(font
+					(size 1.27 1.27)
+				)
+				(hide yes)
+			)
+		)
+		(property "Note-mie" ""
 			(at 220.98 105.41 0)
 			(effects
@@
 			)
 		)
-		(property "MyComment" "x"
+		(property "MyComment" ""
+			(at 82.55 83.82 0)
+			(effects
+				(font
+					(size 1.27 1.27)
+				)
+				(hide yes)
+			)
+		)
+		(property "Note-mie" ""
 			(at 82.55 83.82 0)
 			(effects
@@
 			)
 		)
-		(property "MyComment" "x"
+		(property "MyComment" ""
 			(at 91.44 83.82 0)
 			(effects
+				(font
+					(size 1.27 1.27)
+				)
+				(hide yes)
+			)
+		)
+		(property "Note-mie" ""
+			(at 91.44 83.82 0)
+			(effects
