File: DC_MOTOR_2.kicad_sch (KiCad schematic)
At the start: 17 parts, among them P15 Pad, P17 Pad

Commit message: Aggiornamento PCB
Parts:
- removed U?: TLE9201SG, Package_SO:Infineon_PG-DSO-12-11, symbol chips:TLE9201SG
- added U1: TLE9201SG, Package_SO:Infineon_PG-DSO-12-11, symbol chips:TLE9201SG
- C? (x13), R?: MyComment (none) -> x
- P15, P17: value Pad -> DNP; footprint hellen-one-common:PAD-TH -> Impronte-mie:PAD-TH-senza-serigrafia; MyComment (none) -> x; now not fitted
Connections:
- net 3V3: now also U1.2 (VSO)
- net DIR: now also U1.1 (DIR)
- net DIS: now also U1.11 (DIS)
- net GND: now also U1.10 (SCK), U1.13 (GND), U1.6 (GND), U1.8 (SI), U1.9 (CSN)
- net OUT+: now also U1.7 (OUT2)
- net OUT-: now also U1.5 (OUT1)
- net PWM: now also U1.12 (PWM)
- net PWR: now also U1.4 (VS)

Commit message: Aggiornamento Progetto
Parts:
- C? (x13), R?: MyComment x -> (none)
- P15, P17: value DNP -> Pad; MyComment x -> (none); now fitted
- U1: MyComment x -> (none); now fitted
Changed lines of the file:
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@@
 			)
 		)
-		(property "MyComment" "x"
+		(property "MyComment" ""
+			(at 144.78 83.82 0)
+			(effects
+				(font
+					(size 1.27 1.27)
+				)
+				(hide yes)
+			)
+		)
+		(property "Note-mie" ""
 			(at 144.78 83.82 0)
 			(effects
@@
 			)
 		)
-		(property "MyComment" "x"
+		(property "MyComment" ""
+			(at 118.11 83.82 0)
+			(effects
+				(font
+					(size 1.27 1.27)
+				)
+				(hide yes)
+			)
+		)
+		(property "Note-mie" ""
 			(at 118.11 83.82 0)
 			(effects
@@
 			)
 		)
-		(property "MyComment" "x"
+		(property "MyComment" ""
+			(at 109.22 83.82 0)
+			(effects
+				(font
+					(size 1.27 1.27)
+				)
+				(hide yes)
+			)
+		)
+		(property "Note-mie" ""
 			(at 109.22 83.82 0)
 			(effects
@@
 		(in_bom yes)
 		(on_board yes)
-		(dnp yes)
+		(dnp no)
 		(fields_autoplaced yes)
 		(property "Reference" "U1"
@@
 			)
 		)
-		(property "MyComment" "x"
+		(property "MyComment" ""
+			(at 198.12 93.98 0)
+			(effects
+				(font
+					(size 1.27 1.27)
+				)
+				(hide yes)
+			)
+		)
+		(property "Note-mie" ""
 			(at 198.12 93.98 0)
 			(effects
@@
 			)
 		)
-		(property "MyComment" "x"
+		(property "MyComment" ""
+			(at 219.71 101.6 0)
+			(effects
+				(font
+					(size 1.27 1.27)
+				)
+				(hide yes)
+			)
+		)
+		(property "Note-mie" ""
 			(at 219.71 101.6 0)
 			(effects
@@
 			)
 		)
-		(property "MyComment" "x"
+		(property "MyComment" ""
+			(at 91.44 83.82 0)
+			(effects
+				(font
+					(size 1.27 1.27)
+				)
+				(hide yes)
+			)
+		)
+		(property "Note-mie" ""
 			(at 91.44 83.82 0)
 			(effects
@@
 			)
 		)
-		(property "MyComment" "x"
+		(property "MyComment" ""
+			(at 100.33 83.82 0)
+			(effects
+				(font
+					(size 1.27 1.27)
+				)
+				(hide yes)
+			)
+		)
+		(property "Note-mie" ""
 			(at 100.33 83.82 0)
 			(effects
@@
 			)
 		)
-		(property "MyComment" "x"
+		(property "MyComment" ""
+			(at 73.66 83.82 0)
+			(effects
+				(font
+					(size 1.27 1.27)
+				)
+				(hide yes)
+			)
+		)
+		(property "Note-mie" ""
 			(at 73.66 83.82 0)
 			(effects
@@
 			)
 		)
-		(property "MyComment" "x"
+		(property "MyComment" ""
+			(at 162.56 83.82 0)
+			(effects
+				(font
+					(size 1.27 1.27)
+				)
+				(hide yes)
+			)
+		)
+		(property "Note-mie" ""
 			(at 162.56 83.82 0)
 			(effects
@@
 			)
 		)
-		(property "MyComment" "x"
+		(property "MyComment" ""
+			(at 153.67 83.82 0)
+			(effects
+				(font
+					(size 1.27 1.27)
+				)
+				(hide yes)
+			)
+		)
+		(property "Note-mie" ""
 			(at 153.67 83.82 0)
 			(effects
@@
 			)
 		)
-		(property "MyComment" "x"
+		(property "MyComment" ""
+			(at 135.89 83.82 0)
+			(effects
+				(font
+					(size 1.27 1.27)
+				)
+				(hide yes)
+			)
+		)
+		(property "Note-mie" ""
 			(at 135.89 83.82 0)
 			(effects
@@
 		(in_bom yes)
 		(on_board yes)
-		(dnp yes)
+		(dnp no)
 		(property "Reference" "P15"
 			(at 222.25 107.95 0)
@@
 			)
 		)
-		(property "Value" "DNP"
+		(property "Value" "Pad"
 			(at 220.98 110.49 0)
 			(effects
@@
 			)
 		)
-		(property "MyComment" "x"
+		(property "MyComment" ""
+			(at 220.98 107.95 0)
+			(effects
+				(font
+					(size 1.27 1.27)
+				)
+				(hide yes)
+			)
+		)
+		(property "Note-mie" ""
 			(at 220.98 107.95 0)
 			(effects
@@
 			)
 		)
-		(property "MyComment" "x"
+		(property "MyComment" ""
+			(at 127 83.82 0)
+			(effects
+				(font
+					(size 1.27 1.27)
+				)
+				(hide yes)
+			)
+		)
+		(property "Note-mie" ""
 			(at 127 83.82 0)
 			(effects
@@
 			)
 		)
-		(property "MyComment" "x"
+		(property "MyComment" ""
+			(at 82.55 83.82 0)
+			(effects
+				(font
+					(size 1.27 1.27)
+				)
+				(hide yes)
+			)
+		)
+		(property "Note-mie" ""
 			(at 82.55 83.82 0)
 			(effects
@@
 			)
 		)
-		(property "MyComment" "x"
+		(property "MyComment" ""
+			(at 175.26 92.71 0)
+			(effects
+				(font
+					(size 1.27 1.27)
+				)
+				(hide yes)
+			)
+		)
+		(property "Note-mie" ""
 			(at 175.26 92.71 0)
 			(effects
@@
 			)
 		)
-		(property "MyComment" "x"
+		(property "MyComment" ""
+			(at 175.26 111.76 0)
+			(effects
+				(font
+					(size 1.27 1.27)
+				)
+				(hide yes)
+			)
+		)
+		(property "Note-mie" ""
 			(at 175.26 111.76 0)
 			(effects
@@
 		(in_bom yes)
 		(on_board yes)
-		(dnp yes)
+		(dnp no)
 		(property "Reference" "P17"
 			(at 222.25 105.41 0)
@@
 			)
 		)
-		(property "Value" "DNP"
+		(property "Value" "Pad"
 			(at 220.98 107.95 0)
 			(effects
@@
 			)
 		)
-		(property "MyComment" "x"
+		(property "MyComment" ""
 			(at 220.98 105.41 0)
 			(effects
+				(font
+					(size 1.27 1.27)
+				)
+				(hide yes)
+			)
+		)
+		(property "Note-mie" ""
+			(at 220.98 105.41 0)
+			(effects
