File: 2_DC_MOTOR.kicad_sch (KiCad schematic)
At the start: 34 parts, among them P11 Pad, P12 Pad, P15 Pad, P17 Pad, U1 TLE9201SG, U2 TLE9201SG

Commit message: Riprovo
Parts:
- U2: LCSC C2653438 -> (none); MyComment (none) -> C2653438; Note-mie (none) -> DNP
Changed lines of the file:
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@@
 		(on_board yes)
 		(dnp no)
-		(fields_autoplaced yes)
 		(property "Reference" "U2"
 			(at 170.18 109.22 0)
@@
 			)
 		)
-		(property "LCSC" "C2653438"
+		(property "LCSC" ""
 			(at 175.26 114.3 0)
 			(effects
@@
 			)
 		)
-		(property "MyComment" ""
+		(property "MyComment" "C2653438"
 			(at 175.26 114.3 0)
 			(effects
@@
 			)
 		)
-		(property "Note-mie" ""
-			(at 175.26 114.3 0)
+		(property "Note-mie" "DNP"
+			(at 179.324 111.76 0)
 			(effects
 				(font
 					(size 1.27 1.27)
 				)
-				(hide yes)
 			)
 		)

Commit message: MST01-a1
Parts:
- U1, U2: LCSC (none) -> C2653438; MyComment C2653438 -> Aliexpress; Note-mie DNP -> (none)
Changed lines of the file:
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@@
 			)
 		)
-		(property "LCSC" ""
+		(property "LCSC" "C2653438"
 			(at 175.26 43.18 0)
 			(effects
@@
 			)
 		)
-		(property "MyComment" "C2653438"
+		(property "MyComment" "Aliexpress"
 			(at 175.26 43.18 0)
 			(effects
@@
 			)
 		)
-		(property "Note-mie" "DNP"
+		(property "Note-mie" ""
 			(at 178.816 40.64 0)
 			(effects
@@
 					(size 1.27 1.27)
 				)
+				(hide yes)
 			)
 		)
@@
 			)
 		)
-		(property "LCSC" ""
+		(property "LCSC" "C2653438"
 			(at 175.26 114.3 0)
 			(effects
@@
 			)
 		)
-		(property "MyComment" "C2653438"
+		(property "MyComment" "Aliexpress"
 			(at 175.26 114.3 0)
 			(effects
@@
 			)
 		)
-		(property "Note-mie" "DNP"
+		(property "Note-mie" ""
 			(at 179.324 111.76 0)
 			(effects
@@
 					(size 1.27 1.27)
 				)
-			)
-		)
+				(hide yes)
+			)
+		)

Commit message: MST01-a2
Parts:
- C14, C15, C16, C17, C18, C19, C20, C21, C22, C23, C24, C25, C26, C? (x13), P11, P12, P15, P17, R7, R?: MyComment (none) -> x
Changed lines of the file:
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@@
 			)
 		)
-		(property "MyComment" ""
+		(property "MyComment" "x"
 			(at 104.14 33.02 0)
 			(effects
@@
 			)
 		)
-		(property "MyComment" ""
+		(property "MyComment" "x"
 			(at 68.58 104.14 0)
 			(effects
@@
 			)
 		)
-		(property "MyComment" ""
+		(property "MyComment" "x"
 			(at 86.36 33.02 0)
 			(effects
@@
 			)
 		)
-		(property "MyComment" ""
+		(property "MyComment" "x"
 			(at 130.81 104.14 0)
 			(effects
@@
 			)
 		)
-		(property "MyComment" ""
+		(property "MyComment" "x"
 			(at 130.81 33.02 0)
 			(effects
@@
 			)
 		)
-		(property "MyComment" ""
+		(property "MyComment" "x"
 			(at 152.4 132.08 0)
 			(effects
@@
 			)
 		)
-		(property "MyComment" ""
+		(property "MyComment" "x"
 			(at 113.03 33.02 0)
 			(effects
@@
 			)
 		)
-		(property "MyComment" ""
+		(property "MyComment" "x"
 			(at 152.4 60.96 0)
 			(effects
@@
 			)
 		)
-		(property "MyComment" ""
+		(property "MyComment" "x"
 			(at 198.12 128.27 0)
 			(effects
@@
 			)
 		)
-		(property "MyComment" ""
+		(property "MyComment" "x"
 			(at 50.8 33.02 0)
 			(effects
@@
 			)
 		)
-		(property "MyComment" ""
+		(property "MyComment" "x"
 			(at 139.7 33.02 0)
 			(effects
@@
 			)
 		)
-		(property "MyComment" ""
+		(property "MyComment" "x"
 			(at 50.8 104.14 0)
 			(effects
@@
 			)
 		)
-		(property "MyComment" ""
+		(property "MyComment" "x"
 			(at 77.47 33.02 0)
 			(effects
@@
 			)
 		)
-		(property "MyComment" ""
+		(property "MyComment" "x"
 			(at 121.92 33.02 0)
 			(effects
@@
 			)
 		)
-		(property "MyComment" ""
+		(property "MyComment" "x"
 			(at 198.12 57.15 0)
 			(effects
@@
 			)
 		)
-		(property "MyComment" ""
+		(property "MyComment" "x"
 			(at 152.4 113.03 0)
 			(effects
@@
 			)
 		)
-		(property "MyComment" ""
+		(property "MyComment" "x"
 			(at 95.25 104.14 0)
 			(effects
@@
 			)
 		)
-		(property "MyComment" ""
+		(property "MyComment" "x"
 			(at 139.7 104.14 0)
 			(effects
@@
 			)
 		)
-		(property "MyComment" ""
+		(property "MyComment" "x"
 			(at 196.85 50.8 0)
 			(effects
@@
 			)
 		)
-		(property "MyComment" ""
+		(property "MyComment" "x"
 			(at 95.25 33.02 0)
 			(effects
@@
 			)
 		)
-		(property "MyComment" ""
+		(property "MyComment" "x"
 			(at 104.14 104.14 0)
 			(effects
@@
 			)
 		)
-		(property "MyComment" ""
+		(property "MyComment" "x"
 			(at 59.69 104.14 0)
 			(effects
@@
 			)
 		)
-		(property "MyComment" ""
+		(property "MyComment" "x"
 			(at 198.12 125.73 0)
 			(effects
@@
 			)
 		)
-		(property "MyComment" ""
+		(property "MyComment" "x"
 			(at 152.4 41.91 0)
 			(effects
@@
 			)
 		)
-		(property "MyComment" ""
+		(property "MyComment" "x"
 			(at 121.92 104.14 0)
 			(effects
@@
 			)
 		)
-		(property "MyComment" ""
+		(property "MyComment" "x"
 			(at 113.03 104.14 0)
 			(effects
@@
 			)
 		)
-		(property "MyComment" ""
+		(property "MyComment" "x"
 			(at 198.12 54.61 0)
 			(effects
@@
 			)
 		)
-		(property "MyComment" ""
+		(property "MyComment" "x"
 			(at 196.85 121.92 0)
 			(effects
@@
 			)
 		)
-		(property "MyComment" ""
+		(property "MyComment" "x"
 			(at 86.36 104.14 0)
 			(effects
@@
 			)
 		)
-		(property "MyComment" ""
+		(property "MyComment" "x"
 			(at 59.69 33.02 0)
 			(effects
@@
 			)
 		)
-		(property "MyComment" ""
+		(property "MyComment" "x"
 			(at 77.47 104.14 0)
 			(effects
@@
 			)
 		)
-		(property "MyComment" ""
+		(property "MyComment" "x"
 			(at 68.58 33.02 0)
 			(effects

Commit message: MST01-a5
Parts:
- C14, C15, C16, C17, C18, C19, C20, C21, C22, C23, C24, C25, C26, C? (x13), P11, P12, P15, P17, R7, R?, U1, U2: Verifica file generato da hellen-one *-CPL.csv (none) -> x
