File: IGN6.kicad_sch (KiCad schematic)
At the start: 24 parts

Commit message: Aggiornamento PCB
Parts:
- F10, F5, F6, F7, F8, F9, R14, R7: MyComment (none) -> x
- Q? (x4): value ISL9V3040D3ST -> DNP; MyComment DNP -> x; now not fitted
- Q? (x2): LCSC (none) -> C462128; MyComment DNP -> x
- R14: value 0 -> DNP; MyComment (none) -> x; now not fitted
Changed lines of the file:
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@@
 		(in_bom yes)
 		(on_board yes)
-		(dnp no)
+		(dnp yes)
 		(property "Reference" "Q?"
 			(at 115.7986 124.5616 0)
@@
 			)
 		)
-		(property "Value" "ISL9V3040D3ST"
+		(property "Value" "DNP"
 			(at 115.7986 126.873 0)
 			(effects
@@
 			)
 		)
-		(property "MyComment" "DNP"
+		(property "MyComment" "x"
 			(at 114.3 129.54 0)
 			(effects
@@
 		(in_bom yes)
 		(on_board yes)
-		(dnp no)
+		(dnp yes)
 		(property "Reference" "R14"
 			(at 177.4796 90.0653 0)
@@
 			)
 		)
-		(property "Value" "0"
+		(property "Value" "DNP"
 			(at 177.8 92.71 0)
 			(effects
@@
 		)
 		(property "LCSC" "C25469"
+			(at 182.88 92.71 0)
+			(effects
+				(font
+					(size 1.27 1.27)
+				)
+				(hide yes)
+			)
+		)
+		(property "MyComment" "x"
 			(at 182.88 92.71 0)
 			(effects
@@
 			)
 		)
+		(property "MyComment" "x"
+			(at 186.69 125.73 0)
+			(effects
+				(font
+					(size 1.27 1.27)
+				)
+				(hide yes)
+			)
+		)
 		(pin "1"
 		)
@@
 			)
 		)
+		(property "MyComment" "x"
+			(at 125.73 69.85 0)
+			(effects
+				(font
+					(size 1.27 1.27)
+				)
+				(hide yes)
+			)
+		)
 		(pin "1"
 		)
@@
 		)
 		(property "LCSC" "C25469"
+			(at 182.88 64.77 0)
+			(effects
+				(font
+					(size 1.27 1.27)
+				)
+				(hide yes)
+			)
+		)
+		(property "MyComment" "x"
 			(at 182.88 64.77 0)
 			(effects
@@
 			)
 		)
+		(property "MyComment" "x"
+			(at 172.72 125.73 0)
+			(effects
+				(font
+					(size 1.27 1.27)
+				)
+				(hide yes)
+			)
+		)
 		(pin "1"
 		)
@@
 			)
 		)
+		(property "MyComment" "x"
+			(at 125.73 97.79 0)
+			(effects
+				(font
+					(size 1.27 1.27)
+				)
+				(hide yes)
+			)
+		)
 		(pin "1"
 		)
@@
 			)
 		)
+		(property "MyComment" "x"
+			(at 135.89 64.77 0)
+			(effects
+				(font
+					(size 1.27 1.27)
+				)
+				(hide yes)
+			)
+		)
 		(pin "1"
 		)
@@
 		(property "LCSC" "C369141"
 			(at 186.69 97.79 90)
+			(effects
+				(font
+					(size 1.27 1.27)
+				)
+				(hide yes)
+			)
+		)
+		(property "MyComment" "x"
+			(at 186.69 97.79 0)
 			(effects
 				(font
@@
 		(in_bom yes)
 		(on_board yes)
-		(dnp no)
+		(dnp yes)
 		(property "Reference" "Q?"
 			(at 115.7986 68.6816 0)
@@
 			)
 		)
-		(property "Value" "ISL9V3040D3ST"
+		(property "Value" "DNP"
 			(at 115.7986 70.993 0)
 			(effects
@@
 			)
 		)
-		(property "MyComment" "DNP"
+		(property "MyComment" "x"
 			(at 114.3 73.66 0)
 			(effects
@@
 			)
 		)
+		(property "MyComment" "x"
+			(at 125.73 125.73 0)
+			(effects
+				(font
+					(size 1.27 1.27)
+				)
+				(hide yes)
+			)
+		)
 		(pin "1"
 		)
@@
 		(in_bom yes)
 		(on_board yes)
-		(dnp no)
+		(dnp yes)
 		(property "Reference" "Q?"
 			(at 115.7986 96.6216 0)
@@
 			)
 		)
-		(property "Value" "ISL9V3040D3ST"
+		(property "Value" "DNP"
 			(at 115.7986 98.933 0)
 			(effects
@@
 			)
 		)
-		(property "MyComment" "DNP"
+		(property "MyComment" "x"
 			(at 114.3 101.6 0)
 			(effects
@@
 			)
 		)
+		(property "MyComment" "x"
+			(at 139.7 69.85 0)
+			(effects
+				(font
+					(size 1.27 1.27)
+				)
+				(hide yes)
+			)
+		)
 		(pin "1"
 		)
@@
 		(in_bom yes)
 		(on_board yes)
-		(dnp no)
+		(dnp yes)
 		(property "Reference" "Q?"
 			(at 162.7886 68.6816 0)
@@
 			)
 		)
-		(property "Value" "ISL9V3040D3ST"
+		(property "Value" "DNP"
 			(at 162.7886 70.993 0)
 			(effects
@@
 			)
 		)
-		(property "MyComment" "DNP"
+		(property "MyComment" "x"
 			(at 161.29 73.66 0)
 			(effects
@@
 			)
 		)
+		(property "MyComment" "x"
+			(at 172.72 97.79 0)
+			(effects
+				(font
+					(size 1.27 1.27)
+				)
+				(hide yes)
+			)
+		)
 		(pin "1"
 		)
@@
 			)
 		)
+		(property "MyComment" "x"
+			(at 139.7 97.79 0)
+			(effects
+				(font
+					(size 1.27 1.27)
+				)
+				(hide yes)
+			)
+		)
 		(pin "1"
 		)
@@
 			)
 		)
-		(property "LCSC" ""
+		(property "LCSC" "C462128"
 			(at 167.64 125.73 0)
 			(effects
@@
 			)
 		)
-		(property "MyComment" "DNP"
+		(property "MyComment" "x"
 			(at 161.29 129.54 0)
 			(effects
@@
 		(in_bom yes)
 		(on_board yes)
-		(dnp no)
+		(dnp yes)
 		(property "Reference" "R14"
 			(at 177.4796 118.0053 0)
@@
 			)
 		)
-		(property "Value" "0"
+		(property "Value" "DNP"
 			(at 177.8 120.65 0)
 			(effects
@@
 		)
 		(property "LCSC" "C25469"
+			(at 182.88 120.65 0)
+			(effects
+				(font
+					(size 1.27 1.27)
+				)
+				(hide yes)
+			)
+		)
+		(property "MyComment" "x"
 			(at 182.88 120.65 0)
 			(effects
@@
 			)
 		)
+		(property "MyComment" "x"
+			(at 135.89 92.71 0)
+			(effects
+				(font
+					(size 1.27 1.27)
+				)
+				(hide yes)
+			)
+		)
 		(pin "1"
 		)
@@
 		)
 		(property "LCSC" "C23345"
+			(at 172.72 69.85 0)
+			(effects
+				(font
+					(size 1.27 1.27)
+				)
+				(hide yes)
+			)
+		)
+		(property "MyComment" "x"
 			(at 172.72 69.85 0)
 			(effects
@@
 			)
 		)
+		(property "MyComment" "x"
+			(at 135.89 120.65 0)
+			(effects
+				(font
+					(size 1.27 1.27)
+				)
+				(hide yes)
+			)
+		)
 		(pin "1"
 		)
@@
 			)
 		)
-		(property "LCSC" ""
+		(property "LCSC" "C462128"
 			(at 167.64 97.79 0)
 			(effects
@@
 			)
 		)
-		(property "MyComment" "DNP"
+		(property "MyComment" "x"
 			(at 161.29 101.6 0)
 			(effects
@@
 		(property "LCSC" "C369141"
 			(at 186.69 69.85 90)
+			(effects
+				(font
+					(size 1.27 1.27)
+				)
+				(hide yes)
+			)
+		)
+		(property "MyComment" "x"
+			(at 186.69 69.85 0)
 			(effects
 				(font
@@
 			(effects
 				(font
+					(size 1.27 1.27)
+				)
+				(hide yes)
+			)
+		)
+		(property "MyComment" "x"
+			(at 139.7 125.73 0)
+			(effects
+				(font

Commit message: Aggiornamento Progetto
Parts:
- F10, F5, F6, F7, F8, F9, Q? (x2), R14, R7: MyComment x -> (none)
- Q? (x4): value DNP -> ISL9V3040D3ST; MyComment x -> C462128; Note-mie (none) -> DNP; now fitted
- R14: value DNP -> 0; LCSC C25469 -> (none); MyComment x -> C25469; Note-mie (none) -> DNP; now fitted

Commit message: MST01-a1
Parts:
- Q? (x4): LCSC (none) -> C462128; MyComment C462128 -> (none); Note-mie DNP -> (none)
- R14: LCSC (none) -> C25469; MyComment C25469 -> (none); Note-mie DNP -> (none)
Changed lines of the file:
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@@
 			)
 		)
-		(property "LCSC" ""
+		(property "LCSC" "C462128"
 			(at 120.65 125.73 0)
 			(effects
@@
 			)
 		)
-		(property "MyComment" "C462128"
+		(property "MyComment" ""
 			(at 114.3 129.54 0)
 			(effects
@@
 			)
 		)
-		(property "Note-mie" "DNP"
+		(property "Note-mie" ""
 			(at 111.506 130.556 0)
 			(effects
@@
 					(size 1.27 1.27)
 				)
+				(hide yes)
 			)
 		)
@@
 			)
 		)
-		(property "LCSC" ""
+		(property "LCSC" "C25469"
 			(at 182.88 92.71 0)
 			(effects
@@
 			)
 		)
-		(property "MyComment" "C25469"
+		(property "MyComment" ""
 			(at 182.88 92.71 0)
 			(effects
@@
 			)
 		)
-		(property "Note-mie" "DNP"
+		(property "Note-mie" ""
 			(at 182.626 89.916 0)
 			(effects
@@
 					(size 1.27 1.27)
 				)
+				(hide yes)
 			)
 		)
@@
 			)
 		)
-		(property "LCSC" ""
+		(property "LCSC" "C462128"
 			(at 120.65 71.12 0)
 			(effects
@@
 			)
 		)
-		(property "MyComment" "C462128"
+		(property "MyComment" ""
 			(at 114.3 74.93 0)
 			(effects
@@
 			)
 		)
-		(property "Note-mie" "DNP"
+		(property "Note-mie" ""
 			(at 111.506 74.676 0)
 			(effects
@@
 					(size 1.27 1.27)
 				)
+				(hide yes)
 			)
 		)
@@
 			)
 		)
-		(property "LCSC" ""
+		(property "LCSC" "C462128"
 			(at 120.65 97.79 0)
 			(effects
@@
 			)
 		)
-		(property "MyComment" "C462128"
+		(property "MyComment" ""
 			(at 114.3 101.6 0)
 			(effects
@@
 			)
 		)
-		(property "Note-mie" "DNP"
+		(property "Note-mie" ""
 			(at 112.522 101.346 0)
 			(effects
@@
 					(size 1.27 1.27)
 				)
+				(hide yes)
 			)
 		)
@@
 			)
 		)
-		(property "LCSC" ""
+		(property "LCSC" "C462128"
 			(at 167.64 69.85 0)
 			(effects
@@
 			)
 		)
-		(property "MyComment" "C462128"
+		(property "MyComment" ""
 			(at 161.29 73.66 0)
 			(effects
@@
 			)
 		)
-		(property "Note-mie" "DNP"
+		(property "Note-mie" ""
 			(at 159.258 73.66 0)
 			(effects
@@
 					(size 1.27 1.27)
 				)
+				(hide yes)
 			)
 		)
@@
 					(size 1.27 1.27)
 				)
+				(hide yes)
 			)
 		)
@@
 			)
 		)
-		(property "LCSC" ""
+		(property "LCSC" "C25469"
 			(at 182.88 120.65 0)
 			(effects
@@
 			)
 		)
-		(property "MyComment" "C25469"
+		(property "MyComment" ""
 			(at 182.88 120.65 0)
 			(effects
@@
 			)
 		)
-		(property "Note-mie" "DNP"
+		(property "Note-mie" ""
 			(at 182.626 118.11 0)
 			(effects
@@
 					(size 1.27 1.27)
 				)
+				(hide yes)
 			)
 		)
@@
 					(size 1.27 1.27)
 				)
-			)
-		)
+				(hide yes)
+			)
+		)

Commit message: MST01-a2
Parts:
- F10, F5, F6, F7, F8, F9, Q? (x6), R14, R7: MyComment (none) -> x
Changed lines of the file:
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@@
 			)
 		)
-		(property "MyComment" ""
+		(property "MyComment" "x"
 			(at 114.3 129.54 0)
 			(effects
@@
 			)
 		)
-		(property "MyComment" ""
+		(property "MyComment" "x"
 			(at 182.88 92.71 0)
 			(effects
@@
 			)
 		)
-		(property "MyComment" ""
+		(property "MyComment" "x"
 			(at 186.69 125.73 0)
 			(effects
@@
 			)
 		)
-		(property "MyComment" ""
+		(property "MyComment" "x"
 			(at 125.73 69.85 0)
 			(effects
@@
 			)
 		)
-		(property "MyComment" ""
+		(property "MyComment" "x"
 			(at 182.88 64.77 0)
 			(effects
@@
 			)
 		)
-		(property "MyComment" ""
+		(property "MyComment" "x"
 			(at 172.72 125.73 0)
 			(effects
@@
 			)
 		)
-		(property "MyComment" ""
+		(property "MyComment" "x"
 			(at 125.73 97.79 0)
 			(effects
@@
 			)
 		)
-		(property "MyComment" ""
+		(property "MyComment" "x"
 			(at 135.89 64.77 0)
 			(effects
@@
 			)
 		)
-		(property "MyComment" ""
+		(property "MyComment" "x"
 			(at 186.69 97.79 0)
 			(effects
@@
 			)
 		)
-		(property "MyComment" ""
+		(property "MyComment" "x"
 			(at 114.3 74.93 0)
 			(effects
@@
 			)
 		)
-		(property "MyComment" ""
+		(property "MyComment" "x"
 			(at 125.73 125.73 0)
 			(effects
@@
 			)
 		)
-		(property "MyComment" ""
+		(property "MyComment" "x"
 			(at 114.3 101.6 0)
 			(effects
@@
 			)
 		)
-		(property "MyComment" ""
+		(property "MyComment" "x"
 			(at 139.7 69.85 0)
 			(effects
@@
 			)
 		)
-		(property "MyComment" ""
+		(property "MyComment" "x"
 			(at 161.29 73.66 0)
 			(effects
@@
 			)
 		)
-		(property "MyComment" ""
+		(property "MyComment" "x"
 			(at 172.72 97.79 0)
 			(effects
@@
 			)
 		)
-		(property "MyComment" ""
+		(property "MyComment" "x"
 			(at 139.7 97.79 0)
 			(effects
@@
 			)
 		)
-		(property "MyComment" ""
+		(property "MyComment" "x"
 			(at 161.29 129.54 0)
 			(effects
@@
 			)
 		)
-		(property "MyComment" ""
+		(property "MyComment" "x"
 			(at 182.88 120.65 0)
 			(effects
@@
 			)
 		)
-		(property "MyComment" ""
+		(property "MyComment" "x"
 			(at 135.89 92.71 0)
 			(effects
@@
 			)
 		)
-		(property "MyComment" ""
+		(property "MyComment" "x"
 			(at 172.72 69.85 0)
 			(effects
@@
 			)
 		)
-		(property "MyComment" ""
+		(property "MyComment" "x"
 			(at 135.89 120.65 0)
 			(effects
@@
 			)
 		)
-		(property "MyComment" ""
+		(property "MyComment" "x"
 			(at 161.29 101.6 0)
 			(effects
@@
 			)
 		)
-		(property "MyComment" ""
+		(property "MyComment" "x"
 			(at 186.69 69.85 0)
 			(effects
@@
 			)
 		)
-		(property "MyComment" ""
+		(property "MyComment" "x"
 			(at 139.7 125.73 0)
 			(effects

Commit message: MST01-a5
Parts:
- F10, F5, F6, F7, F8, F9, Q? (x6), R14, R7: Verifica file generato da hellen-one *-CPL.csv (none) -> x
Other:
- moved on the sheet: Q?
