File: INJ6.kicad_sch (KiCad schematic)
At the start: 9 parts, among them U10 VNLD5160TR-E, U11 VNLD5160TR-E, U9 VNLD5160TR-E

Commit message: Aggiornamento PCB
Parts:
- R30, U10, U11, U9: MyComment (none) -> x
Changed lines of the file:
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@@
+			)
+		)
+		(property "MyComment" "x"
+			(at 87.63 52.07 0)
+			(effects
+				(font
+					(size 1.27 1.27)
+				)
+				(hide yes)
 			)
 		)
@@
 			)
 		)
+		(property "MyComment" "x"
+			(at 128.27 88.9 0)
+			(effects
+				(font
+					(size 1.27 1.27)
+				)
+				(hide yes)
+			)
+		)
 		(pin "1"
 		)
@@
 			)
 		)
+		(property "MyComment" "x"
+			(at 87.63 78.74 0)
+			(effects
+				(font
+					(size 1.27 1.27)
+				)
+				(hide yes)
+			)
+		)
 		(pin "1"
 		)
@@
 			)
 		)
+		(property "MyComment" "x"
+			(at 105.41 123.19 0)
+			(effects
+				(font
+					(size 1.27 1.27)
+				)
+				(hide yes)
+			)
+		)
 		(pin "1"
 		)
@@
 			)
 		)
+		(property "MyComment" "x"
+			(at 87.63 107.95 0)
+			(effects
+				(font
+					(size 1.27 1.27)
+				)
+				(hide yes)
+			)
+		)
 		(pin "1"
 		)
@@
 			)
 		)
+		(property "MyComment" "x"
+			(at 105.41 67.31 0)
+			(effects
+				(font
+					(size 1.27 1.27)
+				)
+				(hide yes)
+			)
+		)
 		(pin "1"
 		)
@@
 			)
 		)
+		(property "MyComment" "x"
+			(at 128.27 118.11 0)
+			(effects
+				(font
+					(size 1.27 1.27)
+				)
+				(hide yes)
+			)
+		)
 		(pin "1"
 		)
@@
 			)
 		)
+		(property "MyComment" "x"
+			(at 105.41 93.98 0)
+			(effects
+				(font
+					(size 1.27 1.27)
+				)
+				(hide yes)
+			)
+		)
 		(pin "1"
 		)
@@
 			(at 128.27 62.23 0)
 			(effects
+				(font
+					(size 1.27 1.27)
+				)
+				(hide yes)
+			)
+		)
+		(property "MyComment" "x"
+			(at 128.27 62.23 0)
+			(effects

Commit message: Aggiornamento Progetto
Parts:
- R30, U10, U11, U9: MyComment x -> (none)
Changed lines of the file:
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@@
 			)
 		)
-		(property "MyComment" "x"
+		(property "MyComment" ""
+			(at 87.63 52.07 0)
+			(effects
+				(font
+					(size 1.27 1.27)
+				)
+				(hide yes)
+			)
+		)
+		(property "Note-mie" ""
 			(at 87.63 52.07 0)
 			(effects
@@
 			)
 		)
-		(property "MyComment" "x"
+		(property "MyComment" ""
+			(at 128.27 88.9 0)
+			(effects
+				(font
+					(size 1.27 1.27)
+				)
+				(hide yes)
+			)
+		)
+		(property "Note-mie" ""
 			(at 128.27 88.9 0)
 			(effects
@@
 			)
 		)
-		(property "MyComment" "x"
+		(property "MyComment" ""
+			(at 87.63 78.74 0)
+			(effects
+				(font
+					(size 1.27 1.27)
+				)
+				(hide yes)
+			)
+		)
+		(property "Note-mie" ""
 			(at 87.63 78.74 0)
 			(effects
@@
 			)
 		)
-		(property "MyComment" "x"
+		(property "MyComment" ""
+			(at 105.41 123.19 0)
+			(effects
+				(font
+					(size 1.27 1.27)
+				)
+				(hide yes)
+			)
+		)
+		(property "Note-mie" ""
 			(at 105.41 123.19 0)
 			(effects
@@
 			)
 		)
-		(property "MyComment" "x"
+		(property "MyComment" ""
+			(at 87.63 107.95 0)
+			(effects
+				(font
+					(size 1.27 1.27)
+				)
+				(hide yes)
+			)
+		)
+		(property "Note-mie" ""
 			(at 87.63 107.95 0)
 			(effects
@@
 			)
 		)
-		(property "MyComment" "x"
+		(property "MyComment" ""
+			(at 105.41 67.31 0)
+			(effects
+				(font
+					(size 1.27 1.27)
+				)
+				(hide yes)
+			)
+		)
+		(property "Note-mie" ""
 			(at 105.41 67.31 0)
 			(effects
@@
 			)
 		)
-		(property "MyComment" "x"
+		(property "MyComment" ""
+			(at 128.27 118.11 0)
+			(effects
+				(font
+					(size 1.27 1.27)
+				)
+				(hide yes)
+			)
+		)
+		(property "Note-mie" ""
 			(at 128.27 118.11 0)
 			(effects
@@
 			)
 		)
-		(property "MyComment" "x"
+		(property "MyComment" ""
+			(at 105.41 93.98 0)
+			(effects
+				(font
+					(size 1.27 1.27)
+				)
+				(hide yes)
+			)
+		)
+		(property "Note-mie" ""
 			(at 105.41 93.98 0)
 			(effects
@@
 			)
 		)
-		(property "MyComment" "x"
+		(property "MyComment" ""
 			(at 128.27 62.23 0)
 			(effects
+				(font
+					(size 1.27 1.27)
+				)
+				(hide yes)
+			)
+		)
+		(property "Note-mie" ""
+			(at 128.27 62.23 0)
+			(effects

Commit message: MST01-a2
Parts:
- R30, U10, U11, U9: MyComment (none) -> x
Changed lines of the file:
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@@
 			)
 		)
-		(property "MyComment" ""
+		(property "MyComment" "x"
 			(at 87.63 52.07 0)
 			(effects
@@
 			)
 		)
-		(property "MyComment" ""
+		(property "MyComment" "x"
 			(at 128.27 88.9 0)
 			(effects
@@
 			)
 		)
-		(property "MyComment" ""
+		(property "MyComment" "x"
 			(at 87.63 78.74 0)
 			(effects
@@
 			)
 		)
-		(property "MyComment" ""
+		(property "MyComment" "x"
 			(at 105.41 123.19 0)
 			(effects
@@
 			)
 		)
-		(property "MyComment" ""
+		(property "MyComment" "x"
 			(at 87.63 107.95 0)
 			(effects
@@
 			)
 		)
-		(property "MyComment" ""
+		(property "MyComment" "x"
 			(at 105.41 67.31 0)
 			(effects
@@
 			)
 		)
-		(property "MyComment" ""
+		(property "MyComment" "x"
 			(at 128.27 118.11 0)
 			(effects
@@
 			)
 		)
-		(property "MyComment" ""
+		(property "MyComment" "x"
 			(at 105.41 93.98 0)
 			(effects
@@
 			)
 		)
-		(property "MyComment" ""
+		(property "MyComment" "x"
 			(at 128.27 62.23 0)
 			(effects

Commit message: MST01-a5
Parts:
- R30, U10, U11, U9: Verifica file generato da hellen-one *-CPL.csv (none) -> x
Changed lines of the file:
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@@
+			)
+		)
+		(property "Verifica file generato da hellen-one *-CPL.csv" "x"
+			(at 87.63 52.07 0)
+			(effects
+				(font
+					(size 1.27 1.27)
+				)
+				(hide yes)
 			)
 		)
@@
 			)
 		)
+		(property "Verifica file generato da hellen-one *-CPL.csv" "x"
+			(at 128.27 88.9 0)
+			(effects
+				(font
+					(size 1.27 1.27)
+				)
+				(hide yes)
+			)
+		)
 		(pin "1"
 		)
@@
 			)
 		)
+		(property "Verifica file generato da hellen-one *-CPL.csv" "x"
+			(at 87.63 78.74 0)
+			(effects
+				(font
+					(size 1.27 1.27)
+				)
+				(hide yes)
+			)
+		)
 		(pin "1"
 		)
@@
 			)
 		)
+		(property "Verifica file generato da hellen-one *-CPL.csv" "x"
+			(at 105.41 123.19 0)
+			(effects
+				(font
+					(size 1.27 1.27)
+				)
+				(hide yes)
+			)
+		)
 		(pin "1"
 		)
@@
 			)
 		)
+		(property "Verifica file generato da hellen-one *-CPL.csv" "x"
+			(at 87.63 107.95 0)
+			(effects
+				(font
+					(size 1.27 1.27)
+				)
+				(hide yes)
+			)
+		)
 		(pin "1"
 		)
@@
 			)
 		)
+		(property "Verifica file generato da hellen-one *-CPL.csv" "x"
+			(at 105.41 67.31 0)
+			(effects
+				(font
+					(size 1.27 1.27)
+				)
+				(hide yes)
+			)
+		)
 		(pin "1"
 		)
@@
 			)
 		)
+		(property "Verifica file generato da hellen-one *-CPL.csv" "x"
+			(at 128.27 118.11 0)
+			(effects
+				(font
+					(size 1.27 1.27)
+				)
+				(hide yes)
+			)
+		)
 		(pin "1"
 		)
@@
 			)
 		)
+		(property "Verifica file generato da hellen-one *-CPL.csv" "x"
+			(at 105.41 93.98 0)
+			(effects
+				(font
+					(size 1.27 1.27)
+				)
+				(hide yes)
+			)
+		)
 		(pin "1"
 		)
@@
 			(at 128.27 62.23 0)
 			(effects
+				(font
+					(size 1.27 1.27)
+				)
+				(hide yes)
+			)
+		)
+		(property "Verifica file generato da hellen-one *-CPL.csv" "x"
+			(at 128.27 62.23 0)
+			(effects
