File: LS4.kicad_sch (KiCad schematic)
At the start: 10 parts, among them U7 VNLD5160TR-E, U8 VNLD5160TR-E

Commit message: Aggiornamento PCB
Parts:
- D27, R30, U7, U8: MyComment (none) -> x
Changed lines of the file:
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@@
+			)
+		)
+		(property "MyComment" "x"
+			(at 196.85 95.25 0)
+			(effects
+				(font
+					(size 1.27 1.27)
+				)
+				(hide yes)
 			)
 		)
@@
 			)
 		)
+		(property "MyComment" "x"
+			(at 196.85 121.92 0)
+			(effects
+				(font
+					(size 1.27 1.27)
+				)
+				(hide yes)
+			)
+		)
 		(pin "1"
 		)
@@
 			)
 		)
+		(property "MyComment" "x"
+			(at 156.21 111.76 0)
+			(effects
+				(font
+					(size 1.27 1.27)
+				)
+				(hide yes)
+			)
+		)
 		(pin "1"
 		)
@@
 			)
 		)
+		(property "MyComment" "x"
+			(at 100.33 123.19 0)
+			(effects
+				(font
+					(size 1.27 1.27)
+				)
+				(hide yes)
+			)
+		)
 		(pin "1"
 		)
@@
 			)
 		)
+		(property "MyComment" "x"
+			(at 100.33 107.95 0)
+			(effects
+				(font
+					(size 1.27 1.27)
+				)
+				(hide yes)
+			)
+		)
 		(pin "1"
 		)
@@
 			)
 		)
+		(property "MyComment" "x"
+			(at 100.33 81.28 0)
+			(effects
+				(font
+					(size 1.27 1.27)
+				)
+				(hide yes)
+			)
+		)
 		(pin "1"
 		)
@@
 			)
 		)
+		(property "MyComment" "x"
+			(at 156.21 85.09 0)
+			(effects
+				(font
+					(size 1.27 1.27)
+				)
+				(hide yes)
+			)
+		)
 		(pin "1"
 		)
@@
 			)
 		)
+		(property "MyComment" "x"
+			(at 100.33 96.52 0)
+			(effects
+				(font
+					(size 1.27 1.27)
+				)
+				(hide yes)
+			)
+		)
 		(pin "1"
 		)
@@
 			)
 		)
+		(property "MyComment" "x"
+			(at 171.45 127 0)
+			(effects
+				(font
+					(size 1.27 1.27)
+				)
+				(hide yes)
+			)
+		)
 		(pin "1"
 		)
@@
 			(at 171.45 100.33 0)
 			(effects
+				(font
+					(size 1.27 1.27)
+				)
+				(hide yes)
+			)
+		)
+		(property "MyComment" "x"
+			(at 171.45 100.33 0)
+			(effects

Commit message: Aggiornamento Progetto
Parts:
- D27, R30, U7, U8: MyComment x -> (none)
Changed lines of the file:
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@@
 			)
 		)
-		(property "MyComment" "x"
+		(property "MyComment" ""
+			(at 196.85 95.25 0)
+			(effects
+				(font
+					(size 1.27 1.27)
+				)
+				(hide yes)
+			)
+		)
+		(property "Note-mie" ""
 			(at 196.85 95.25 0)
 			(effects
@@
 			)
 		)
-		(property "MyComment" "x"
+		(property "MyComment" ""
+			(at 196.85 121.92 0)
+			(effects
+				(font
+					(size 1.27 1.27)
+				)
+				(hide yes)
+			)
+		)
+		(property "Note-mie" ""
 			(at 196.85 121.92 0)
 			(effects
@@
 			)
 		)
-		(property "MyComment" "x"
+		(property "MyComment" ""
+			(at 156.21 111.76 0)
+			(effects
+				(font
+					(size 1.27 1.27)
+				)
+				(hide yes)
+			)
+		)
+		(property "Note-mie" ""
 			(at 156.21 111.76 0)
 			(effects
@@
 			)
 		)
-		(property "MyComment" "x"
+		(property "MyComment" ""
+			(at 100.33 123.19 0)
+			(effects
+				(font
+					(size 1.27 1.27)
+				)
+				(hide yes)
+			)
+		)
+		(property "Note-mie" ""
 			(at 100.33 123.19 0)
 			(effects
@@
 			)
 		)
-		(property "MyComment" "x"
+		(property "MyComment" ""
+			(at 100.33 107.95 0)
+			(effects
+				(font
+					(size 1.27 1.27)
+				)
+				(hide yes)
+			)
+		)
+		(property "Note-mie" ""
 			(at 100.33 107.95 0)
 			(effects
@@
 			)
 		)
-		(property "MyComment" "x"
+		(property "MyComment" ""
+			(at 100.33 81.28 0)
+			(effects
+				(font
+					(size 1.27 1.27)
+				)
+				(hide yes)
+			)
+		)
+		(property "Note-mie" ""
 			(at 100.33 81.28 0)
 			(effects
@@
 			)
 		)
-		(property "MyComment" "x"
+		(property "MyComment" ""
+			(at 156.21 85.09 0)
+			(effects
+				(font
+					(size 1.27 1.27)
+				)
+				(hide yes)
+			)
+		)
+		(property "Note-mie" ""
 			(at 156.21 85.09 0)
 			(effects
@@
 			)
 		)
-		(property "MyComment" "x"
+		(property "MyComment" ""
+			(at 100.33 96.52 0)
+			(effects
+				(font
+					(size 1.27 1.27)
+				)
+				(hide yes)
+			)
+		)
+		(property "Note-mie" ""
 			(at 100.33 96.52 0)
 			(effects
@@
 			)
 		)
-		(property "MyComment" "x"
+		(property "MyComment" ""
+			(at 171.45 127 0)
+			(effects
+				(font
+					(size 1.27 1.27)
+				)
+				(hide yes)
+			)
+		)
+		(property "Note-mie" ""
 			(at 171.45 127 0)
 			(effects
@@
 			)
 		)
-		(property "MyComment" "x"
+		(property "MyComment" ""
 			(at 171.45 100.33 0)
 			(effects
+				(font
+					(size 1.27 1.27)
+				)
+				(hide yes)
+			)
+		)
+		(property "Note-mie" ""
+			(at 171.45 100.33 0)
+			(effects

Commit message: MST01-a2
Parts:
- D27, R30, U7, U8: MyComment (none) -> x
Changed lines of the file:
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@@
 			)
 		)
-		(property "MyComment" ""
+		(property "MyComment" "x"
 			(at 196.85 95.25 0)
 			(effects
@@
 			)
 		)
-		(property "MyComment" ""
+		(property "MyComment" "x"
 			(at 196.85 121.92 0)
 			(effects
@@
 			)
 		)
-		(property "MyComment" ""
+		(property "MyComment" "x"
 			(at 156.21 111.76 0)
 			(effects
@@
 			)
 		)
-		(property "MyComment" ""
+		(property "MyComment" "x"
 			(at 100.33 123.19 0)
 			(effects
@@
 			)
 		)
-		(property "MyComment" ""
+		(property "MyComment" "x"
 			(at 100.33 107.95 0)
 			(effects
@@
 			)
 		)
-		(property "MyComment" ""
+		(property "MyComment" "x"
 			(at 100.33 81.28 0)
 			(effects
@@
 			)
 		)
-		(property "MyComment" ""
+		(property "MyComment" "x"
 			(at 156.21 85.09 0)
 			(effects
@@
 			)
 		)
-		(property "MyComment" ""
+		(property "MyComment" "x"
 			(at 100.33 96.52 0)
 			(effects
@@
 			)
 		)
-		(property "MyComment" ""
+		(property "MyComment" "x"
 			(at 171.45 127 0)
 			(effects
@@
 			)
 		)
-		(property "MyComment" ""
+		(property "MyComment" "x"
 			(at 171.45 100.33 0)
 			(effects

Commit message: MST01-a5
Parts:
- D27, R30, U7, U8: Verifica file generato da hellen-one *-CPL.csv (none) -> x
Changed lines of the file:
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@@
+			)
+		)
+		(property "Verifica file generato da hellen-one *-CPL.csv" "x"
+			(at 196.85 95.25 0)
+			(effects
+				(font
+					(size 1.27 1.27)
+				)
+				(hide yes)
 			)
 		)
@@
 			)
 		)
+		(property "Verifica file generato da hellen-one *-CPL.csv" "x"
+			(at 196.85 121.92 0)
+			(effects
+				(font
+					(size 1.27 1.27)
+				)
+				(hide yes)
+			)
+		)
 		(pin "1"
 		)
@@
 			)
 		)
+		(property "Verifica file generato da hellen-one *-CPL.csv" "x"
+			(at 156.21 111.76 0)
+			(effects
+				(font
+					(size 1.27 1.27)
+				)
+				(hide yes)
+			)
+		)
 		(pin "1"
 		)
@@
 			)
 		)
+		(property "Verifica file generato da hellen-one *-CPL.csv" "x"
+			(at 100.33 123.19 0)
+			(effects
+				(font
+					(size 1.27 1.27)
+				)
+				(hide yes)
+			)
+		)
 		(pin "1"
 		)
@@
 			)
 		)
+		(property "Verifica file generato da hellen-one *-CPL.csv" "x"
+			(at 100.33 107.95 0)
+			(effects
+				(font
+					(size 1.27 1.27)
+				)
+				(hide yes)
+			)
+		)
 		(pin "1"
 		)
@@
 			)
 		)
+		(property "Verifica file generato da hellen-one *-CPL.csv" "x"
+			(at 100.33 81.28 0)
+			(effects
+				(font
+					(size 1.27 1.27)
+				)
+				(hide yes)
+			)
+		)
 		(pin "1"
 		)
@@
 			)
 		)
+		(property "Verifica file generato da hellen-one *-CPL.csv" "x"
+			(at 156.21 85.09 0)
+			(effects
+				(font
+					(size 1.27 1.27)
+				)
+				(hide yes)
+			)
+		)
 		(pin "1"
 		)
@@
 			)
 		)
+		(property "Verifica file generato da hellen-one *-CPL.csv" "x"
+			(at 100.33 96.52 0)
+			(effects
+				(font
+					(size 1.27 1.27)
+				)
+				(hide yes)
+			)
+		)
 		(pin "1"
 		)
@@
 			)
 		)
+		(property "Verifica file generato da hellen-one *-CPL.csv" "x"
+			(at 171.45 127 0)
+			(effects
+				(font
+					(size 1.27 1.27)
+				)
+				(hide yes)
+			)
+		)
 		(pin "1"
 		)
@@
 			(at 171.45 100.33 0)
 			(effects
+				(font
+					(size 1.27 1.27)
+				)
+				(hide yes)
+			)
+		)
+		(property "Verifica file generato da hellen-one *-CPL.csv" "x"
+			(at 171.45 100.33 0)
+			(effects
