File: MAP.kicad_sch (KiCad schematic)
At the start: 4 parts, among them U12 MPXH6400A

Commit message: Aggiornamento PCB
Parts:
- C2, U12: MyComment (none) -> x
- H1, H2: MyComment (none) -> x; now not fitted
Changed lines of the file:
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@@
+			)
+		)
+		(property "MyComment" "x"
+			(at 140.97 85.09 0)
+			(effects
+				(font
+					(size 1.27 1.27)
+				)
+				(hide yes)
 			)
 		)
@@
 		(in_bom no)
 		(on_board yes)
-		(dnp no)
+		(dnp yes)
 		(fields_autoplaced yes)
 		(property "Reference" "H1"
@@
 		)
 		(property "Description" "Mounting Hole without connection"
+			(at 124.46 109.22 0)
+			(effects
+				(font
+					(size 1.27 1.27)
+				)
+				(hide yes)
+			)
+		)
+		(property "MyComment" "x"
 			(at 124.46 109.22 0)
 			(effects
@@
 		(in_bom no)
 		(on_board yes)
-		(dnp no)
+		(dnp yes)
 		(fields_autoplaced yes)
 		(property "Reference" "H2"
@@
 		)
 		(property "Description" "Mounting Hole without connection"
+			(at 148.59 109.22 0)
+			(effects
+				(font
+					(size 1.27 1.27)
+				)
+				(hide yes)
+			)
+		)
+		(property "MyComment" "x"
 			(at 148.59 109.22 0)
 			(effects
@@
 			(at 165.1 92.71 0)
 			(effects
+				(font
+					(size 1.27 1.27)
+				)
+				(hide yes)
+			)
+		)
+		(property "MyComment" "x"
+			(at 165.1 92.71 0)
+			(effects

Commit message: Aggiornamento Progetto
Parts:
- C2, U12: MyComment x -> (none)
- H1, H2: MyComment x -> (none); now fitted
Changed lines of the file:
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@@
 			)
 		)
-		(property "MyComment" "x"
+		(property "MyComment" ""
+			(at 140.97 85.09 0)
+			(effects
+				(font
+					(size 1.27 1.27)
+				)
+				(hide yes)
+			)
+		)
+		(property "Note-mie" ""
 			(at 140.97 85.09 0)
 			(effects
@@
 		(in_bom no)
 		(on_board yes)
-		(dnp yes)
+		(dnp no)
 		(fields_autoplaced yes)
 		(property "Reference" "H1"
@@
 			)
 		)
-		(property "MyComment" "x"
+		(property "MyComment" ""
+			(at 124.46 109.22 0)
+			(effects
+				(font
+					(size 1.27 1.27)
+				)
+				(hide yes)
+			)
+		)
+		(property "Note-mie" ""
 			(at 124.46 109.22 0)
 			(effects
@@
 		(in_bom no)
 		(on_board yes)
-		(dnp yes)
+		(dnp no)
 		(fields_autoplaced yes)
 		(property "Reference" "H2"
@@
 			)
 		)
-		(property "MyComment" "x"
+		(property "MyComment" ""
+			(at 148.59 109.22 0)
+			(effects
+				(font
+					(size 1.27 1.27)
+				)
+				(hide yes)
+			)
+		)
+		(property "Note-mie" ""
 			(at 148.59 109.22 0)
 			(effects
@@
 			)
 		)
-		(property "MyComment" "x"
+		(property "MyComment" ""
 			(at 165.1 92.71 0)
 			(effects
+				(font
+					(size 1.27 1.27)
+				)
+				(hide yes)
+			)
+		)
+		(property "Note-mie" ""
+			(at 165.1 92.71 0)
+			(effects

Commit message: MST01-a2
Parts:
- C2, H1, H2, U12: MyComment (none) -> x
Changed lines of the file:
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@@
 			)
 		)
-		(property "MyComment" ""
+		(property "MyComment" "x"
 			(at 140.97 85.09 0)
 			(effects
@@
 			)
 		)
-		(property "MyComment" ""
+		(property "MyComment" "x"
 			(at 124.46 109.22 0)
 			(effects
@@
 			)
 		)
-		(property "MyComment" ""
+		(property "MyComment" "x"
 			(at 148.59 109.22 0)
 			(effects
@@
 			)
 		)
-		(property "MyComment" ""
+		(property "MyComment" "x"
 			(at 165.1 92.71 0)
 			(effects

Commit message: MST01-a5
Parts:
- C2, H1, H2, U12: Verifica file generato da hellen-one *-CPL.csv (none) -> x
Changed lines of the file:
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@@
+			)
+		)
+		(property "Verifica file generato da hellen-one *-CPL.csv" "x"
+			(at 140.97 85.09 0)
+			(effects
+				(font
+					(size 1.27 1.27)
+				)
+				(hide yes)
 			)
 		)
@@
 			)
 		)
+		(property "Verifica file generato da hellen-one *-CPL.csv" "x"
+			(at 124.46 109.22 0)
+			(effects
+				(font
+					(size 1.27 1.27)
+				)
+				(hide yes)
+			)
+		)
 		(instances
 			(project ""
@@
 			)
 		)
+		(property "Verifica file generato da hellen-one *-CPL.csv" "x"
+			(at 148.59 109.22 0)
+			(effects
+				(font
+					(size 1.27 1.27)
+				)
+				(hide yes)
+			)
+		)
 		(instances
 			(project "MST-01A"
@@
 			(at 165.1 92.71 0)
 			(effects
+				(font
+					(size 1.27 1.27)
+				)
+				(hide yes)
+			)
+		)
+		(property "Verifica file generato da hellen-one *-CPL.csv" "x"
+			(at 165.1 92.71 0)
+			(effects
