File: MST01.kicad_sch (KiCad schematic)
At the start: 46 parts, among them J1 Conn_01x35, J1 USB_B_Mini, J2 Conn_01x35, J3 Conn_01x04_Pin, J6 Conn_01x05, M1 Module-power_12and5V-0.2, M3 Module-knock-0.2, M3 Module-vr-discrete-0.5, M4 Module-vr-max9924-0.1, M5 Module-wbo-0.5, M6 Module:mega-mcu100/0.3, M7 Module-can-0.1, P1 Pad, P10 Pad, P2 Pad, P3 Pad, P4 Pad, P5 Pad, P6 Pad, P7 Pad, P8 Pad, P9 Pad, U5 JDY-33-mio

Commit message: Aggiornamento
Connections:
- net P9: now reaches J1.31 (Pin_31), P9.1 (Pin_1)
- net nReset: now reaches J6.5 (Pin_5), M5.W5 (nReset)
- net SWDIO: now reaches J6.4 (Pin_4), M5.W6 (SWDIO)
- net SWCLK: now reaches J6.2 (Pin_2), M5.W7 (SWCLK)
- net V33_OUT: now reaches J6.1 (Pin_1), M5.W8 (V33_OUT)
- net P10: now reaches J1.26 (Pin_26), P10.1 (Pin_1)
- net P2: now reaches J2.33 (Pin_33), P2.1 (Pin_1)
- net P1: now reaches J2.32 (Pin_32), P1.1 (Pin_1)
Other:
- moved on the sheet: J6, P1, P2
Changed lines of the file:
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@@
 	(wire
 		(pts
-			(xy 71.12 167.64) (xy 68.58 167.64)
+			(xy 82.55 167.64) (xy 68.58 167.64)
 		)
 		(stroke
@@
 	(wire
 		(pts
-			(xy 220.98 90.17) (xy 229.87 90.17)
+			(xy 220.98 90.17) (xy 246.38 90.17)
 		)
 		(stroke
@@
 		)
 	)
+	(wire
+		(pts
+			(xy 246.38 85.09) (xy 229.87 85.09)
+		)
+		(stroke
+			(width 0)
+			(type default)
+		)
+	)
 	(bus
 		(pts
@@
 	(wire
 		(pts
-			(xy 220.98 80.01) (xy 229.87 80.01)
+			(xy 220.98 80.01) (xy 246.38 80.01)
 		)
 		(stroke
@@
 	(wire
 		(pts
-			(xy 71.12 165.1) (xy 68.58 165.1)
+			(xy 82.55 165.1) (xy 68.58 165.1)
 		)
 		(stroke
@@
 	(wire
 		(pts
-			(xy 220.98 82.55) (xy 229.87 82.55)
+			(xy 220.98 82.55) (xy 246.38 82.55)
 		)
 		(stroke
@@
 	(wire
 		(pts
-			(xy 222.25 87.63) (xy 229.87 87.63)
+			(xy 222.25 87.63) (xy 246.38 87.63)
 		)
 		(stroke
@@
 	)
 	(circle
-		(center 234.95 85.09)
+		(center 251.46 85.09)
 		(radius 8.132)
 		(stroke
@@
 		)
 	)
+	(label "P10"
+		(at 71.12 248.92 0)
+		(effects
+			(font
+				(size 1.27 1.27)
+			)
+			(justify left bottom)
+		)
+	)
 	(label "OUT_LS_HOT2"
 		(at 189.23 143.51 0)
@@
 		)
 	)
+	(label "P2"
+		(at 71.12 167.64 0)
+		(effects
+			(font
+				(size 1.27 1.27)
+			)
+			(justify left bottom)
+		)
+	)
 	(label "LS4"
 		(at 223.52 191.77 0)
@@
 		)
 	)
+	(label "V33_OUT"
+		(at 232.41 80.01 0)
+		(effects
+			(font
+				(size 1.27 1.27)
+			)
+			(justify left bottom)
+		)
+	)
 	(label "OUT_DC2-"
 		(at 71.12 185.42 0)
@@
 		)
 	)
+	(label "SWDIO"
+		(at 232.41 87.63 0)
+		(effects
+			(font
+				(size 1.27 1.27)
+			)
+			(justify left bottom)
+		)
+	)
 	(label "VR_DISCRETE_THR"
 		(at 248.92 201.93 180)
@@
 		)
 	)
+	(label "P1"
+		(at 71.12 165.1 0)
+		(effects
+			(font
+				(size 1.27 1.27)
+			)
+			(justify left bottom)
+		)
+	)
 	(label "CLT"
 		(at 71.12 129.54 0)
@@
 		)
 	)
+	(label "nReset"
+		(at 232.41 90.17 0)
+		(effects
+			(font
+				(size 1.27 1.27)
+			)
+			(justify left bottom)
+		)
+	)
 	(label "WBO_Rtrim"
 		(at 71.12 210.82 0)
@@
 		)
 	)
+	(label "P9"
+		(at 71.12 261.62 0)
+		(effects
+			(font
+				(size 1.27 1.27)
+			)
+			(justify left bottom)
+		)
+	)
 	(label "AUX2"
 		(at 248.92 240.03 180)
@@
 		)
 	)
+	(label "GND"
+		(at 232.41 85.09 0)
+		(effects
+			(font
+				(size 1.27 1.27)
+			)
+			(justify left bottom)
+		)
+	)
 	(label "OUT_IGN5"
 		(at 189.23 129.54 0)
@@
 		)
 	)
+	(label "SWCLK"
+		(at 232.41 82.55 0)
+		(effects
+			(font
+				(size 1.27 1.27)
+			)
+			(justify left bottom)
+		)
+	)
 	(label "WBO_Ip"
 		(at 71.12 236.22 0)
@@
 	(symbol
 		(lib_id "Connector_Generic:Conn_01x05")
-		(at 234.95 85.09 0)
+		(at 251.46 85.09 0)
 		(unit 1)
 		(exclude_from_sim no)
@@
 		(fields_autoplaced yes)
 		(property "Reference" "J6"
-			(at 237.49 83.8199 0)
+			(at 254 83.8199 0)
 			(effects
 				(font
@@
 		)
 		(property "Value" "Conn_01x05"
-			(at 237.49 86.3599 0)
+			(at 254 86.3599 0)
 			(effects
 				(font
@@
 		)
 		(property "Footprint" "Connector_PinHeader_2.54mm:PinHeader_1x05_P2.54mm_Vertical"
-			(at 234.95 85.09 0)
+			(at 251.46 85.09 0)
 			(effects
 				(font
@@
 		)
 		(property "Datasheet" "~"
-			(at 234.95 85.09 0)
+			(at 251.46 85.09 0)
 			(effects
 				(font
@@
 		)
 		(property "Description" "Generic connector, single row, 01x05, script generated (kicad-library-utils/schlib/autogen/connector/)"
-			(at 234.95 85.09 0)
+			(at 251.46 85.09 0)
 			(effects
 				(font
@@
 	(symbol
 		(lib_id "hellen-one-common:Pad")
-		(at 76.2 167.64 0)
+		(at 87.63 167.64 0)
 		(unit 1)
 		(exclude_from_sim no)
@@
 		(dnp no)
 		(property "Reference" "P2"
-			(at 77.724 167.386 0)
+			(at 89.154 167.386 0)
 			(effects
 				(font
@@
 		)
 		(property "Value" "Pad"
-			(at 76.2 170.18 0)
+			(at 87.63 170.18 0)
 			(effects
 				(font
@@
 		)
 		(property "Footprint" "hellen-one-common:PAD-TH"
-			(at 76.2 171.45 0)
+			(at 87.63 171.45 0)
 			(effects
 				(font
@@
 		)
 		(property "Datasheet" "~"
-			(at 76.2 167.64 0)
+			(at 87.63 167.64 0)
 			(effects
 				(font
@@
 		)
 		(property "Description" ""
-			(at 76.2 167.64 0)
+			(at 87.63 167.64 0)
 			(effects
 				(font
@@
 	(symbol
 		(lib_id "hellen-one-common:Pad")
-		(at 76.2 165.1 0)
+		(at 87.63 165.1 0)
 		(unit 1)
 		(exclude_from_sim no)
@@
 		(dnp no)
 		(property "Reference" "P1"
-			(at 77.724 164.846 0)
+			(at 89.154 164.846 0)
 			(effects
 				(font
@@
 		)
 		(property "Value" "Pad"
-			(at 76.2 167.64 0)
+			(at 87.63 167.64 0)
 			(effects
 				(font
@@
 		)
 		(property "Footprint" "hellen-one-common:PAD-TH"
-			(at 76.2 168.91 0)
+			(at 87.63 168.91 0)
 			(effects
 				(font
@@
 		)
 		(property "Datasheet" "~"
-			(at 76.2 165.1 0)
+			(at 87.63 165.1 0)
 			(effects
 				(font
@@
 		)
 		(property "Description" ""
-			(at 76.2 165.1 0)
+			(at 87.63 165.1 0)
 			(effects
 				(font
@@
 				)
 			)
-			(project "MST-01A"
+			(project "MST01"
 				(path "/ac264c30-3e9a-4be2-b97a-9949b68bd497"
 					(page "2")
@@
 		)
 		(instances
-			(project "MST-01A"
+			(project "MST01"
 				(path "/ac264c30-3e9a-4be2-b97a-9949b68bd497"
 					(page "10")
@@
 		)
 		(instances
-			(project "MST-01A"
+			(project "MST01"
 				(path "/ac264c30-3e9a-4be2-b97a-9949b68bd497"
 					(page "8")
@@
 		)
 		(instances
-			(project "MST-01A"
+			(project "MST01"
 				(path "/ac264c30-3e9a-4be2-b97a-9949b68bd497"
 					(page "9")
@@
 		)
 		(instances
-			(project "MST-01A"
+			(project "MST01"
 				(path "/ac264c30-3e9a-4be2-b97a-9949b68bd497"
 					(page "3")
@@
 				)
 			)
-			(project "MST-01A"
+			(project "MST01"
 				(path "/ac264c30-3e9a-4be2-b97a-9949b68bd497"
 					(page "4")
@@
 		)
 		(instances
-			(project "MST-01A"
+			(project "MST01"
 				(path "/ac264c30-3e9a-4be2-b97a-9949b68bd497"
 					(page "6")
@@
 		)
 		(instances
-			(project "MST-01A"
+			(project "MST01"
 				(path "/ac264c30-3e9a-4be2-b97a-9949b68bd497"
 					(page "9")

Commit message: Aggiornamento Progetto
Parts:
- removed J1, J2: Conn_01x35, ampseal:ampseal-35-mia, symbol Connector_Generic:Conn_01x35
- added J1, J2: Conn_01x36, ampseal:ampseal-35-mia-con-pad-GND, symbol Connector_Generic:Conn_01x36
Connections:
- net +12V: now also J1.24 (Pin_24)
- net +5VP: now also J2.21 (Pin_21), J2.22 (Pin_22), J2.34 (Pin_34)
- net 12V_KEY: now also J1.25 (Pin_25)
- net AUX1: now also J2.26 (Pin_26)
- net AUX2: now also J2.15 (Pin_15)
- net AUX3: now also J2.25 (Pin_25)
- net BUTTON1: now also J2.16 (Pin_16)
- net BUTTON2: now also J2.27 (Pin_27)
- net BUTTON3: now also J2.13 (Pin_13)
- net CAN1+: now also J1.35 (Pin_35)
- net CAN1-: now also J1.34 (Pin_34)
- net CAN2+: now also J2.1 (Pin_1)
- net CAN2-: now also J2.2 (Pin_2)
- net CLT: now also J2.18 (Pin_18)
- net EGT+: now also J2.12 (Pin_12)
- net EGT-: now also J2.35 (Pin_35)
- net FLEX: now also J2.8 (Pin_8)
- net GND: now also J1.27 (Pin_27), J1.33 (Pin_33), J1.36 (Pin_36), J2.19 (Pin_19), J2.36 (Pin_36)
- net GNDA: now also J2.29 (Pin_29), J2.30 (Pin_30), J2.31 (Pin_31)
- net HALL1: now also J2.5 (Pin_5)
- net HALL2: now also J2.4 (Pin_4)
- net HALL3: now also J2.24 (Pin_24)
- net IAT: now also J2.20 (Pin_20)
- net IMP_VR_DISCRETE+: now also J2.23 (Pin_23)
- net IMP_VR_DISCRETE-: now also J2.11 (Pin_11)
- net IMP_VR_MAX9924+: now also J2.10 (Pin_10)
- net IMP_VR_MAX9924-: now also J2.9 (Pin_9)
- net IN_KNOCK_RAW: now also J2.3 (Pin_3)
- net MAP: now also J2.7 (Pin_7)
- net OUT_DC1+: now also J1.14 (Pin_14)
- net OUT_DC1-: now also J1.13 (Pin_13)
- net OUT_DC2+: now also J1.2 (Pin_2)
- net OUT_DC2-: now also J1.1 (Pin_1)
- net OUT_IGN1: now also J1.10 (Pin_10)
- net OUT_IGN2: now also J1.9 (Pin_9)
- net OUT_IGN3: now also J1.32 (Pin_32)
- net OUT_IGN4: now also J1.30 (Pin_30)
- net OUT_IGN5: now also J1.29 (Pin_29)
- net OUT_IGN6: now also J1.28 (Pin_28)
- net OUT_INJ1: now also J1.5 (Pin_5)
- net OUT_INJ2: now also J1.17 (Pin_17)
- net OUT_INJ3: now also J1.18 (Pin_18)
- net OUT_INJ4: now also J1.6 (Pin_6)
- net OUT_INJ5: now also J1.7 (Pin_7)
- net OUT_INJ6: now also J1.19 (Pin_19)
- net OUT_LS1: now also J1.15 (Pin_15)
- net OUT_LS2: now also J1.3 (Pin_3)
- net OUT_LS3: now also J1.16 (Pin_16)
- net OUT_LS4: now also J1.4 (Pin_4)
- net OUT_LS_HOT1: now also J1.20 (Pin_20)
- net OUT_LS_HOT2: now also J1.8 (Pin_8)
- net P1: now also J2.32 (Pin_32)
- net P10: now also J1.26 (Pin_26)
- net P2: now also J2.33 (Pin_33)
- net P9: now also J1.31 (Pin_31)
- net PPS1: now also J2.28 (Pin_28)
- net PPS2: now also J2.14 (Pin_14)
- net TPS1: now also J2.17 (Pin_17)
- net TPS2: now also J2.6 (Pin_6)
- net WBO_Heater: now also J1.23 (Pin_23)
- net WBO_Ip: now also J1.21 (Pin_21)
- net WBO_Rtrim: now also J1.11 (Pin_11)
- net WBO_Un: now also J1.12 (Pin_12)
- net WBO_Vm: now also J1.22 (Pin_22)

Commit message: Aggiornamento PCB
Parts:
- BT1, C3, D10, F6, J1, R30, R38, R4: MyComment (none) -> x
- G1, G2, G3, G4, M1, M3, M4, M5, M6, M7, R38, R39, R41: MyComment (none) -> x; now not fitted
- J1: value Conn_01x36 -> DNP; LCSC (none) -> 776231-1; MyComment (none) -> Aliexpress; now not fitted
- J2: value Conn_01x36 -> DNP; LCSC (none) -> 776231-4; MyComment (none) -> Aliexpress; now not fitted
- J3: LCSC (none) -> C5305780; MyComment (none) -> Ci sono
- J6: value Conn_01x05 -> DNP; MyComment (none) -> Ci sono; now not fitted
- P1, P2, P3, P4, P5, P6, P7, P8, P9: value Pad -> DNP; MyComment (none) -> x; now not fitted
- P10: value Pad -> DNP; footprint hellen-one-common:PAD-TH -> Impronte-mie:PAD-TH-senza-serigrafia; MyComment (none) -> x; now not fitted
- R30: value 0 -> DNP; MyComment DNP -> x; now not fitted
- R30: value 4.7k -> DNP; MyComment DNP -> x; now not fitted
- U5: MyComment (none) -> Aliexpress; now not fitted
Connections:
- net GND: now also J1.32 (Pin_32); no longer J1.33 (Pin_33)
- net OUT_DC1+: now also J1.1 (Pin_1); no longer J1.14 (Pin_14)
- net OUT_DC1-: now also J1.2 (Pin_2); no longer J1.13 (Pin_13)
- net OUT_DC2+: now also J1.13 (Pin_13); no longer J1.2 (Pin_2)
- net OUT_DC2-: now also J1.14 (Pin_14); no longer J1.1 (Pin_1)
- net OUT_IGN3: now also J1.33 (Pin_33); no longer J1.32 (Pin_32)
Other:
- sheet DC Driver 1: file DC_MOTOR_0.1.kicad_sch -> DC_MOTOR_1.kicad_sch
- sheet DC Driver 2: file DC_MOTOR_0.1.kicad_sch -> DC_MOTOR_2.kicad_sch

Commit message: Aggiornamento Progetto
Parts:
- BT1, C3, D10, F6, J1, R30, R38, R4: MyComment x -> (none)
- G1, G2, G3, G4, M1, M3, M4, M5, M6, M7: MyComment x -> (none); now fitted
- J1: value DNP -> AMPSeal-35-verticale-nero; LCSC 776231-1 -> (none); MyComment Aliexpress -> 776231-1 Aliexpress; Note-mie (none) -> DNP; now fitted
- J2: value DNP -> AMPSeal-35-verticale-bianco; LCSC 776231-4 -> (none); MyComment Aliexpress -> 776231-4 Aliexpress; Note-mie (none) -> DNP; now fitted
- J3: MyComment Ci sono -> (none)
- J6: value DNP -> Conn_01x05_Pin; Note-mie (none) -> DNP; now fitted
- P1, P10, P2, P3, P4, P5, P6, P7, P8, P9: value DNP -> Pad; MyComment x -> (none); now fitted
- R30: value DNP -> 0; MyComment x -> C21189; Note-mie (none) -> DNP; now fitted
- R30: value DNP -> 4.7k; MyComment x -> C23162; Note-mie (none) -> DNP; now fitted
- R38, R39, R41: value DNP -> 10k; MyComment x -> C17414; Note-mie (none) -> DNP; now fitted
- U5: value JDY-33-mio -> JDY-33; LCSC C9900001612 -> (none); MyComment Aliexpress -> C9900001612 Aliexpress; Note-mie (none) -> DNP; now fitted

Commit message: Aggiornamento Progetto
Connections:
- net 2 DC Driver/PWR renamed 2 DC Driver/PWR1
- net DC Driver 2/PWR renamed 2 DC Driver/PWR2
Other:
- sheet DC Driver 1 renamed 2 DC Driver
- removed sheet DC Driver 2
- sheet 2 DC Driver: file DC_MOTOR_1.kicad_sch -> 2_DC_MOTOR.kicad_sch
- sheet 2 DC Driver ports: added DIR1, DIR2, DIS1, DIS2, OUT1+, OUT1-, OUT2+, OUT2-, PWM1, PWM2, PWR1, PWR2; removed DIR, DIS, OUT+, OUT-, PWM, PWR

Commit message: MST01-a1
Parts:
- J1: LCSC (none) -> 776231-1; MyComment 776231-1 Aliexpress -> Aliexpress; Note-mie DNP -> (none)
- J2: LCSC (none) -> 776231-4; MyComment 776231-4 Aliexpress -> Aliexpress; Note-mie DNP -> (none)
- J6: MyComment Ci sono -> (none); Note-mie DNP -> (none)
- R30: LCSC (none) -> C21189; MyComment C21189 -> (none); Note-mie DNP -> (none)
- R30: LCSC (none) -> C23162; MyComment C23162 -> (none); Note-mie DNP -> (none)
- R38, R39, R41: LCSC (none) -> C17414; MyComment C17414 -> (none); Note-mie DNP -> (none)
- U5: LCSC (none) -> C9900001612; MyComment C9900001612 Aliexpress -> Aliexpress; Note-mie DNP -> (none)
Changed lines of the file:
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@@
 			)
 		)
-		(property "LCSC" ""
+		(property "LCSC" "C9900001612"
 			(at 357.886 191.262 0)
 			(effects
@@
 			)
 		)
-		(property "MyComment" "C9900001612   Aliexpress"
+		(property "MyComment" "Aliexpress"
 			(at 349.25 208.28 0)
 			(effects
@@
 			)
 		)
-		(property "Note-mie" "DNP"
-			(at 365.506 194.31 0)
-			(effects
-				(font
-					(size 1.27 1.27)
-				)
-			)
-		)
 		(pin "19"
 		)
@@
 			)
 		)
-		(property "LCSC" ""
+		(property "LCSC" "C21189"
 			(at 219.71 265.43 0)
 			(effects
@@
 			)
 		)
-		(property "MyComment" "C21189"
+		(property "MyComment" ""
 			(at 224.79 265.43 0)
 			(effects
@@
 			)
 		)
-		(property "Note-mie" "DNP"
+		(property "Note-mie" ""
 			(at 224.536 268.478 0)
 			(effects
@@
 					(size 1.27 1.27)
 				)
+				(hide yes)
 			)
 		)
@@
 			)
 		)
-		(property "MyComment" "Ci sono"
+		(property "MyComment" ""
 			(at 251.46 85.09 0)
 			(effects
@@
 			)
 		)
-		(property "Note-mie" "DNP"
+		(property "Note-mie" ""
 			(at 261.874 88.646 0)
 			(effects
@@
 					(size 1.27 1.27)
 				)
+				(hide yes)
 			)
 		)
@@
 			)
 		)
-		(property "MyComment" "776231-4    Aliexpress"
+		(property "MyComment" "Aliexpress"
 			(at 63.5 129.54 0)
 			(effects
@@
 			)
 		)
-		(property "LCSC" ""
+		(property "LCSC" "776231-4"
 			(at 63.5 129.54 0)
 			(effects
@@
 			)
 		)
-		(property "Note-mie" "DNP"
+		(property "Note-mie" ""
 			(at 58.42 129.54 0)
 			(effects
@@
 					(size 1.27 1.27)
 				)
+				(hide yes)
 			)
 		)
@@
 			)
 		)
-		(property "MyComment" "776231-1    Aliexpress"
+		(property "MyComment" "Aliexpress"
 			(at 63.5 228.6 0)
 			(effects
@@
 			)
 		)
-		(property "LCSC" ""
+		(property "LCSC" "776231-1"
 			(at 63.5 228.6 0)
 			(effects
@@
 			)
 		)
-		(property "Note-mie" "DNP"
+		(property "Note-mie" ""
 			(at 58.674 223.774 0)
 			(effects
@@
 					(size 1.27 1.27)
 				)
+				(hide yes)
 			)
 		)
@@
 			)
 		)
-		(property "LCSC" ""
+		(property "LCSC" "C23162"
 			(at 127 313.69 0)
 			(effects
@@
 			)
 		)
-		(property "MyComment" "C23162"
+		(property "MyComment" ""
 			(at 132.08 313.69 0)
 			(effects
@@
 			)
 		)
-		(property "Note-mie" "DNP"
+		(property "Note-mie" ""
 			(at 127.508 315.976 0)
 			(effects
@@
 					(size 1.27 1.27)
 				)
+				(hide yes)
 			)
 		)
@@
 			)
 		)
-		(property "LCSC" ""
+		(property "LCSC" "C17414"
 			(at 311.15 398.78 0)
 			(effects
@@
 			)
 		)
-		(property "MyComment" "C17414"
+		(property "MyComment" ""
 			(at 311.15 398.78 0)
 			(effects
@@
 			)
 		)
-		(property "Note-mie" "DNP"
+		(property "Note-mie" ""
 			(at 308.61 396.494 0)
 			(effects
@@
 					(size 1.27 1.27)
 				)
+				(hide yes)
 			)
 		)
@@
 			)
 		)
-		(property "LCSC" ""
+		(property "LCSC" "C17414"
 			(at 311.15 393.7 0)
 			(effects
@@
 			)
 		)
-		(property "MyComment" "C17414"
+		(property "MyComment" ""
 			(at 311.15 393.7 0)
 			(effects
@@
 			)
 		)
-		(property "Note-mie" "DNP"
+		(property "Note-mie" ""
 			(at 308.356 391.414 0)
 			(effects
@@
 					(size 1.27 1.27)
 				)
+				(hide yes)
 			)
 		)
@@
 			)
 		)
-		(property "LCSC" ""
+		(property "LCSC" "C17414"
 			(at 311.15 388.62 0)
 			(effects
@@
 			)
 		)
-		(property "MyComment" "C17414"
+		(property "MyComment" ""
 			(at 311.15 388.62 0)
 			(effects
@@
 			)
 		)
-		(property "Note-mie" "DNP"
+		(property "Note-mie" ""
 			(at 308.356 386.334 0)
 			(effects
@@
 					(size 1.27 1.27)
 				)
+				(hide yes)
 			)
 		)

Commit message: MST01-a2
Parts:
- removed M1: Module-power_12and5V-0.2, hellen-one-power_12and5V-0.2:power_12and5V, symbol hellen-one-power_12and5V:Module-power_12and5V-0.2
- added M1: Module-power_12and5V-0.3, hellen-one-power_12and5V-0.3:power_12and5V, symbol hellen-one-power_12and5V-0.3:Module-power_12and5V-0.3
- BT1, C3, D10, F6, G1, G2, G3, G4, J1, J3, J6, M3, M4, M5, M6, M7, P1, P10, P2, P3, P4, P5, P6, P7, P8, P9, R30, R38, R39, R4, R41: MyComment (none) -> x
Connections:
- net +12V_RAW: now also M1.V1 (V12_PERM), M1.V3 (V12_RAW)
- net +5V: now also M1.E4 (V5)
- net +5VP: now also M1.V4 (5VP)
- net GND: now also M1.S1 (GND)
- net IN_VIGN: now also M1.V2 (IN_VIGN)
- net PWR_EN: now also M1.E5 (EN_5VP)
- net VBAT: now also M1.E1 (VBAT)
- net VIGN: now also M1.E3 (VIGN)
- net at R4.1: now also M1.E6 (PG_5VP)

Commit message: MST01-a5
Parts:
- C3, D10, F6, G1, G2, G3, G4, J1, J2, J3, J6, P1, P10, P2, P3, P4, P5, P6, P7, P8, P9, R30, R38, R39, R4, R41, U5: Verifica file generato da hellen-one *-CPL.csv (none) -> x
