File: MST01.kicad_sch (KiCad schematic)
At the start: 46 parts, among them J1 AMPSeal-35-verticale-nero, J1 USB_B_Mini, J2 AMPSeal-35-verticale-bianco, J3 Conn_01x04_Pin, J6 Conn_01x05_Pin, M1 Module-power_12and5V-0.3, M3 Module-knock-0.2, M3 Module-vr-discrete-0.5, M4 Module-vr-max9924-0.1, M5 Module-wbo-0.5, M6 Module:mega-mcu100/0.3, M7 Module-can-0.1, P1 Pad, P10 Pad, P2 Pad, P3 Pad, P4 Pad, P5 Pad, P6 Pad, P7 Pad, P8 Pad, P9 Pad, U5 JDY-33

Commit message: aggiornamento
Parts:
- M1, M3, M4, M5, M6, M7: Verifica file generato da hellen-one *-CPL.csv (none) -> x
Changed lines of the file:
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@@
 			)
 		)
-		(property "Verifica file generato da hellen-one *-CPL.csv" ""
+		(property "Verifica file generato da hellen-one *-CPL.csv" "x"
 			(at 154.94 298.45 0)
 			(effects
@@
 			)
 		)
-		(property "Verifica file generato da hellen-one *-CPL.csv" ""
+		(property "Verifica file generato da hellen-one *-CPL.csv" "x"
 			(at 154.94 334.01 0)
 			(effects
@@
 			)
 		)
-		(property "Verifica file generato da hellen-one *-CPL.csv" ""
+		(property "Verifica file generato da hellen-one *-CPL.csv" "x"
 			(at 248.92 138.43 0)
 			(effects
@@
 			)
 		)
-		(property "Verifica file generato da hellen-one *-CPL.csv" ""
+		(property "Verifica file generato da hellen-one *-CPL.csv" "x"
 			(at 153.67 372.11 0)
 			(effects
@@
 			)
 		)
-		(property "Verifica file generato da hellen-one *-CPL.csv" ""
+		(property "Verifica file generato da hellen-one *-CPL.csv" "x"
 			(at 153.67 257.81 0)
 			(effects
@@
 			)
 		)
-		(property "Verifica file generato da hellen-one *-CPL.csv" ""
+		(property "Verifica file generato da hellen-one *-CPL.csv" "x"
 			(at 213.36 67.31 0)
 			(effects
@@
 			)
 		)
-		(property "Verifica file generato da hellen-one *-CPL.csv" ""
+		(property "Verifica file generato da hellen-one *-CPL.csv" "x"
 			(at 271.78 92.71 0)
 			(effects
