File: egt.kicad_sch (KiCad schematic)
At the start: 9 parts, among them U4 MAX31855KASA

Commit message: Aggiornamento PCB
Parts:
- C? (x5), D8, L1, L2, U4: MyComment (none) -> x
Connections:
- net T-Filtrato: now reaches C?.1, C?.2, D8.1 (K), L2.2, U4.2 (T-)
- net T+Filtrato: now reaches C?.2, C?.2, D8.2 (K), L1.2, U4.3 (T+)
Changed lines of the file:
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@@
+		)
+	)
+	(label "T-Filtrato"
+		(at 125.73 95.25 0)
+		(effects
+			(font
+				(size 1.27 1.27)
+			)
+			(justify left bottom)
+		)
+	)
+	(label "T+Filtrato"
+		(at 127 87.63 0)
+		(effects
+			(font
+				(size 1.27 1.27)
+			)
+			(justify left bottom)
 		)
 	)
@@
 			)
 		)
+		(property "MyComment" "x"
+			(at 135.89 101.6 0)
+			(effects
+				(font
+					(size 1.27 1.27)
+				)
+				(hide yes)
+			)
+		)
 		(pin "1"
 		)
@@
 			)
 		)
+		(property "MyComment" "x"
+			(at 166.37 92.71 0)
+			(effects
+				(font
+					(size 1.27 1.27)
+				)
+				(hide yes)
+			)
+		)
 		(pin "1"
 		)
@@
 		)
 		(property "LCSC" "C15849"
+			(at 189.23 73.66 0)
+			(effects
+				(font
+					(size 1.27 1.27)
+				)
+				(hide yes)
+			)
+		)
+		(property "MyComment" "x"
 			(at 189.23 73.66 0)
 			(effects
@@
 			)
 		)
+		(property "MyComment" "x"
+			(at 151.13 101.6 0)
+			(effects
+				(font
+					(size 1.27 1.27)
+				)
+				(hide yes)
+			)
+		)
 		(pin "1"
 		)
@@
 			)
 		)
+		(property "MyComment" "x"
+			(at 119.38 101.6 0)
+			(effects
+				(font
+					(size 1.27 1.27)
+				)
+				(hide yes)
+			)
+		)
 		(pin "3"
 		)
@@
 			)
 		)
+		(property "MyComment" "x"
+			(at 176.53 73.66 0)
+			(effects
+				(font
+					(size 1.27 1.27)
+				)
+				(hide yes)
+			)
+		)
 		(pin "1"
 		)
@@
 			)
 		)
+		(property "MyComment" "x"
+			(at 106.68 95.25 0)
+			(effects
+				(font
+					(size 1.27 1.27)
+				)
+				(hide yes)
+			)
+		)
 		(pin "1"
 		)
@@
 			)
 		)
+		(property "MyComment" "x"
+			(at 142.24 91.44 0)
+			(effects
+				(font
+					(size 1.27 1.27)
+				)
+				(hide yes)
+			)
+		)
 		(pin "1"
 		)
@@
 			(effects
 				(font
+					(size 1.27 1.27)
+				)
+				(hide yes)
+			)
+		)
+		(property "MyComment" "x"
+			(at 106.68 87.63 0)
+			(effects
+				(font

Commit message: Aggiornamento Progetto
Parts:
- C? (x5), D8, L1, L2, U4: MyComment x -> (none)
Changed lines of the file:
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@@
 			)
 		)
-		(property "MyComment" "x"
+		(property "MyComment" ""
+			(at 135.89 101.6 0)
+			(effects
+				(font
+					(size 1.27 1.27)
+				)
+				(hide yes)
+			)
+		)
+		(property "Note-mie" ""
 			(at 135.89 101.6 0)
 			(effects
@@
 			)
 		)
-		(property "MyComment" "x"
+		(property "MyComment" ""
+			(at 166.37 92.71 0)
+			(effects
+				(font
+					(size 1.27 1.27)
+				)
+				(hide yes)
+			)
+		)
+		(property "Note-mie" ""
 			(at 166.37 92.71 0)
 			(effects
@@
 			)
 		)
-		(property "MyComment" "x"
+		(property "MyComment" ""
+			(at 189.23 73.66 0)
+			(effects
+				(font
+					(size 1.27 1.27)
+				)
+				(hide yes)
+			)
+		)
+		(property "Note-mie" ""
 			(at 189.23 73.66 0)
 			(effects
@@
 			)
 		)
-		(property "MyComment" "x"
+		(property "MyComment" ""
+			(at 151.13 101.6 0)
+			(effects
+				(font
+					(size 1.27 1.27)
+				)
+				(hide yes)
+			)
+		)
+		(property "Note-mie" ""
 			(at 151.13 101.6 0)
 			(effects
@@
 			)
 		)
-		(property "MyComment" "x"
+		(property "MyComment" ""
+			(at 119.38 101.6 0)
+			(effects
+				(font
+					(size 1.27 1.27)
+				)
+				(hide yes)
+			)
+		)
+		(property "Note-mie" ""
 			(at 119.38 101.6 0)
 			(effects
@@
 			)
 		)
-		(property "MyComment" "x"
+		(property "MyComment" ""
+			(at 176.53 73.66 0)
+			(effects
+				(font
+					(size 1.27 1.27)
+				)
+				(hide yes)
+			)
+		)
+		(property "Note-mie" ""
 			(at 176.53 73.66 0)
 			(effects
@@
 			)
 		)
-		(property "MyComment" "x"
+		(property "MyComment" ""
+			(at 106.68 95.25 0)
+			(effects
+				(font
+					(size 1.27 1.27)
+				)
+				(hide yes)
+			)
+		)
+		(property "Note-mie" ""
 			(at 106.68 95.25 0)
 			(effects
@@
 			)
 		)
-		(property "MyComment" "x"
+		(property "MyComment" ""
+			(at 142.24 91.44 0)
+			(effects
+				(font
+					(size 1.27 1.27)
+				)
+				(hide yes)
+			)
+		)
+		(property "Note-mie" ""
 			(at 142.24 91.44 0)
 			(effects
@@
 			)
 		)
-		(property "MyComment" "x"
+		(property "MyComment" ""
 			(at 106.68 87.63 0)
 			(effects
+				(font
+					(size 1.27 1.27)
+				)
+				(hide yes)
+			)
+		)
+		(property "Note-mie" ""
+			(at 106.68 87.63 0)
+			(effects

Commit message: MST01-a1
Changed lines of the file:
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@@
 		(dnp no)
 		(property "Reference" "U4"
-			(at 168.5641 80.01 0)
+			(at 156.21 77.47 0)
 			(effects
 				(font
@@
 		)
 		(property "Value" "MAX31855KASA"
-			(at 168.5641 82.55 0)
+			(at 151.892 81.026 0)
 			(effects
 				(font

Commit message: MST01-a2
Parts:
- C? (x5), D8, L1, L2, U4: MyComment (none) -> x
Changed lines of the file:
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@@
 			)
 		)
-		(property "MyComment" ""
+		(property "MyComment" "x"
 			(at 135.89 101.6 0)
 			(effects
@@
 			)
 		)
-		(property "MyComment" ""
+		(property "MyComment" "x"
 			(at 166.37 92.71 0)
 			(effects
@@
 			)
 		)
-		(property "MyComment" ""
+		(property "MyComment" "x"
 			(at 189.23 73.66 0)
 			(effects
@@
 			)
 		)
-		(property "MyComment" ""
+		(property "MyComment" "x"
 			(at 151.13 101.6 0)
 			(effects
@@
 			)
 		)
-		(property "MyComment" ""
+		(property "MyComment" "x"
 			(at 119.38 101.6 0)
 			(effects
@@
 			)
 		)
-		(property "MyComment" ""
+		(property "MyComment" "x"
 			(at 176.53 73.66 0)
 			(effects
@@
 			)
 		)
-		(property "MyComment" ""
+		(property "MyComment" "x"
 			(at 106.68 95.25 0)
 			(effects
@@
 			)
 		)
-		(property "MyComment" ""
+		(property "MyComment" "x"
 			(at 142.24 91.44 0)
 			(effects
@@
 			)
 		)
-		(property "MyComment" ""
+		(property "MyComment" "x"
 			(at 106.68 87.63 0)
 			(effects

Commit message: MST01-a5
Parts:
- C? (x5), D8, L1, L2, U4: Verifica file generato da hellen-one *-CPL.csv (none) -> x
Changed lines of the file:
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@@
+			)
+		)
+		(property "Verifica file generato da hellen-one *-CPL.csv" "x"
+			(at 135.89 101.6 0)
+			(effects
+				(font
+					(size 1.27 1.27)
+				)
+				(hide yes)
 			)
 		)
@@
 			)
 		)
+		(property "Verifica file generato da hellen-one *-CPL.csv" "x"
+			(at 166.37 92.71 0)
+			(effects
+				(font
+					(size 1.27 1.27)
+				)
+				(hide yes)
+			)
+		)
 		(pin "1"
 		)
@@
 		)
 		(property "Note-mie" ""
+			(at 189.23 73.66 0)
+			(effects
+				(font
+					(size 1.27 1.27)
+				)
+				(hide yes)
+			)
+		)
+		(property "Verifica file generato da hellen-one *-CPL.csv" "x"
 			(at 189.23 73.66 0)
 			(effects
@@
 			)
 		)
+		(property "Verifica file generato da hellen-one *-CPL.csv" "x"
+			(at 151.13 101.6 0)
+			(effects
+				(font
+					(size 1.27 1.27)
+				)
+				(hide yes)
+			)
+		)
 		(pin "1"
 		)
@@
 			)
 		)
+		(property "Verifica file generato da hellen-one *-CPL.csv" "x"
+			(at 119.38 101.6 0)
+			(effects
+				(font
+					(size 1.27 1.27)
+				)
+				(hide yes)
+			)
+		)
 		(pin "3"
 		)
@@
 			)
 		)
+		(property "Verifica file generato da hellen-one *-CPL.csv" "x"
+			(at 176.53 73.66 0)
+			(effects
+				(font
+					(size 1.27 1.27)
+				)
+				(hide yes)
+			)
+		)
 		(pin "1"
 		)
@@
 			)
 		)
+		(property "Verifica file generato da hellen-one *-CPL.csv" "x"
+			(at 106.68 95.25 0)
+			(effects
+				(font
+					(size 1.27 1.27)
+				)
+				(hide yes)
+			)
+		)
 		(pin "1"
 		)
@@
 			)
 		)
+		(property "Verifica file generato da hellen-one *-CPL.csv" "x"
+			(at 142.24 91.44 0)
+			(effects
+				(font
+					(size 1.27 1.27)
+				)
+				(hide yes)
+			)
+		)
 		(pin "1"
 		)
@@
 			(at 106.68 87.63 0)
 			(effects
+				(font
+					(size 1.27 1.27)
+				)
+				(hide yes)
+			)
+		)
+		(property "Verifica file generato da hellen-one *-CPL.csv" "x"
+			(at 106.68 87.63 0)
+			(effects
